File: hardware/kicad/nofilterbooth/camera.sch (KiCad schematic (older format))
At the start: 62 parts

Commit message: clean
Parts:
- C1, C2, C3, C_ATTINY1, C_AUX1, C_AUX2, C_CEILING1, C_FLASH1, C_RADIO1, C_START1: symbol Device:CP -> nofilterbooth:CP-Device
- CONN_AUX1, CONN_BATT1, CONN_FLASH1, CONN_SW_SCISSOR1, CONN_SW_SHUTTER1: symbol Connector_Generic:Conn_01x02 -> nofilterbooth:Conn_01x02-Connector_Generic
- CONN_CEILING1, CONN_MARQUEE_WS2811, CONN_SW_PAP1, CONN_SW_PAP2, CONN_SW_PAP3, CONN_SW_PAP4: symbol Connector_Generic:Conn_01x03 -> nofilterbooth:Conn_01x03-Connector_Generic
- CONN_COIN1, CONN_LUXSENSOR1, CONN_SEGMENT1, CONN_START1, CONN_STEP_PAPER1, CONN_STEP_SCISSOR1, CONN_STEP_SHUTTER1: symbol Connector_Generic:Conn_01x04 -> nofilterbooth:Conn_01x04-Connector_Generic
- CONN_MATRIX1: symbol Connector_Generic:Conn_01x05 -> nofilterbooth:Conn_01x05-Connector_Generic
- C_COIN1: symbol Device:C -> nofilterbooth:C-Device
- C_LUXSENSOR1, C_MATRIX1, C_SEGMENT1: footprint (none) -> Capacitor_THT:C_Disc_D3.0mm_W1.6mm_P2.50mm; symbol Device:C -> nofilterbooth:C-Device
- DRV_PAPER1, DRV_SCISSOR1, DRV_SHUTTER1: symbol pololu_breakout_drv8825:Pololu_Breakout_DRV8825 -> nofilterbooth:Pololu_Breakout_DRV8825
- LED_SW_PAPER1, LED_SW_PAPER2, LED_SW_PAPER3, LED_SW_PAPER4, LED_SW_SCISSOR1, LED_SW_SHUTTER1, LED_SW_START1: symbol Device:LED_Small -> nofilterbooth:LED_Small-Device
- MEGA_CAMERA1: footprint MEGA2560PRO-EMBED:MEGA2560PRO-EMBED -> footprints:MEGA2560PRO-EMBED; symbol MEGA2560PRO-EMBED:MEGA2560PRO-EMBED -> nofilterbooth:MEGA2560PRO-EMBED
- Q_AUX1, Q_FLASH1, Q_START1: symbol Transistor_BJT:TIP120 -> nofilterbooth:TIP120-Transistor_BJT
- R_BATT1, R_BATT2, R_FLASH1, R_FLASH2, R_MARQUEE1, R_START1, R_SW_PAPER1, R_SW_PAPER2, R_SW_PAPER3, R_SW_PAPER4, R_SW_SCISSOR1, R_SW_SHUTTER1, R_SW_START1: symbol Device:R_Small -> nofilterbooth:R_Small-Device
- U_MARQUEE1: symbol MCU_Microchip_ATtiny:ATtiny85-20PU -> nofilterbooth:ATtiny85-20PU-MCU_Microchip_ATtiny
- U_RADIO1: symbol RF:NRF24L01_Breakout -> nofilterbooth:NRF24L01_Breakout-RF
Connections:
- net labels added: +12V-power, +5V-power, GND-power
