File: hardware/kicad/nofilterbooth/nofilterbooth.kicad_pcb (KiCad board)
At the start: 2 copper layers, 47 parts, among them U1 NRF24L01_Breakout

Commit message: clean
Parts:
- added CONN_CEILING1: JST_XH3, Connector_JST:JST_XH_S3B-XH-A_1x03_P2.50mm_Horizontal, F.Cu at (107.7, 147.0)
- added CONN_COIN1: Conn_01x04, Connector_JST:JST_XH_S4B-XH-A_1x04_P2.50mm_Horizontal, F.Cu at (60.4, 165.3)
- added CONN_LUXSENSOR1: Conn_01x04, Connector_JST:JST_XH_S4B-XH-A_1x04_P2.50mm_Horizontal, F.Cu at (76.3, 160.5)
- added CONN_MATRIX1: Conn_01x05, Connector_JST:JST_XH_S5B-XH-A_1x05_P2.50mm_Horizontal, F.Cu at (60.4, 147.0)
- added CONN_SEGMENT1: Conn_01x04, Connector_JST:JST_XH_S4B-XH-A_1x04_P2.50mm_Horizontal, F.Cu at (93.2, 147.0)
- added CONN_START1: Conn_01x04, Connector_JST:JST_XH_S4B-XH-A_1x04_P2.50mm_Horizontal, F.Cu at (90.7, 160.5)
- added C_ATTINY1: 0.1uF, Capacitor_THT:CP_Radial_D10.0mm_P5.00mm, F.Cu at (74.9, 176.5)
- added C_CEILING1: 100uF, Capacitor_THT:CP_Radial_D10.0mm_P5.00mm, F.Cu at (86.7, 176.5)
- added C_MATRIX1: 100nF, Capacitor_THT:C_Disc_D3.0mm_W1.6mm_P2.50mm, F.Cu at (149.9, 165.1)
- added C_RADIO1: 10uF, Capacitor_THT:CP_Radial_D10.0mm_P5.00mm, F.Cu at (105.2, 163.0)
- added C_START1: 100uF, Capacitor_THT:CP_Radial_D10.0mm_P5.00mm, F.Cu at (119.7, 149.4)
- added LED_SW_START1: LED_Small, LED_THT:LED_D3.0mm, F.Cu at (58.6, 178.3)
- added Q_START1: TIP120, Package_TO_SOT_THT:TO-220-3_Vertical, F.Cu at (77.1, 152.3)
- added R_START1: 2.2k 1/2W, Resistor_THT:R_Axial_DIN0309_L9.0mm_D3.2mm_P12.70mm_Horizontal, F.Cu at (58.5, 159.6)
- added R_SW_START1: 560ohm 1/2W, Resistor_THT:R_Axial_DIN0309_L9.0mm_D3.2mm_P12.70mm_Horizontal, F.Cu at (75.5, 146.0)
- C_AUX2: value 1000uF -> 1000uF 16v
- renumbered U1 to U_RADIO1
Connections:
- DRV_PAPER1 pad 2: (no net) -> Net-(DRV_PAPER1-Pad2)
- DRV_SCISSOR1 pad 2: (no net) -> Net-(DRV_SCISSOR1-Pad2)
- DRV_SHUTTER1 pad 2: (no net) -> Net-(DRV_SHUTTER1-Pad2)
- MEGA_CAMERA1 pad A0: (no net) -> Net-(MEGA_CAMERA1-PadA0)
- MEGA_CAMERA1 pad A1: (no net) -> Net-(MEGA_CAMERA1-PadA1)
- MEGA_CAMERA1 pad A10: (no net) -> Net-(MEGA_CAMERA1-PadA10)
- MEGA_CAMERA1 pad A11: (no net) -> Net-(MEGA_CAMERA1-PadA11)
- MEGA_CAMERA1 pad A12: (no net) -> Net-(MEGA_CAMERA1-PadA12)
- MEGA_CAMERA1 pad A13: (no net) -> Net-(MEGA_CAMERA1-PadA13)
- MEGA_CAMERA1 pad A14: (no net) -> Net-(MEGA_CAMERA1-PadA14)
- MEGA_CAMERA1 pad A2: (no net) -> Net-(MEGA_CAMERA1-PadA2)
- MEGA_CAMERA1 pad A3: (no net) -> Net-(MEGA_CAMERA1-PadA3)
- MEGA_CAMERA1 pad A4: (no net) -> Net-(MEGA_CAMERA1-PadA4)
- MEGA_CAMERA1 pad A5: (no net) -> Net-(MEGA_CAMERA1-PadA5)
- MEGA_CAMERA1 pad A6: (no net) -> Net-(MEGA_CAMERA1-PadA6)
- MEGA_CAMERA1 pad A7: (no net) -> Net-(MEGA_CAMERA1-PadA7)
- MEGA_CAMERA1 pad A8: (no net) -> Net-(MEGA_CAMERA1-PadA8)
- MEGA_CAMERA1 pad A9: (no net) -> Net-(MEGA_CAMERA1-PadA9)
- MEGA_CAMERA1 pad AREF: (no net) -> Net-(MEGA_CAMERA1-PadAREF)
- MEGA_CAMERA1 pad D10: (no net) -> LED_MATRIX_SCL_PIN
- MEGA_CAMERA1 pad D11: (no net) -> LED_MATRIX_CS_PIN
- MEGA_CAMERA1 pad D12: (no net) -> LED_MATRIX_SDI_PIN
- MEGA_CAMERA1 pad D13: (no net) -> Net-(MEGA_CAMERA1-PadD13)
- MEGA_CAMERA1 pad D14: (no net) -> LED_START_BTN_PIN
- MEGA_CAMERA1 pad D15: (no net) -> START_BTN_PIN
- MEGA_CAMERA1 pad D16: (no net) -> /Paper/SERIAL_RX2
- MEGA_CAMERA1 pad D17: (no net) -> /Camera/SERIAL_RX2
- MEGA_CAMERA1 pad D18: (no net) -> Net-(MEGA_CAMERA1-PadD18)
- MEGA_CAMERA1 pad D19: (no net) -> Net-(MEGA_CAMERA1-PadD19)
- MEGA_CAMERA1 pad D2: ENABLE_MARQUEE -> RADIO_INTERRUPT
- MEGA_CAMERA1 pad D20: (no net) -> SDA_PIN
- MEGA_CAMERA1 pad D21: (no net) -> SCL_PIN
- MEGA_CAMERA1 pad D22: (no net) -> Net-(MEGA_CAMERA1-PadD22)
- MEGA_CAMERA1 pad D23: (no net) -> /Camera/ORDER_INTERRUPT_PIN
- MEGA_CAMERA1 pad D24: (no net) -> Net-(MEGA_CAMERA1-PadD24)
- MEGA_CAMERA1 pad D25: (no net) -> Net-(MEGA_CAMERA1-PadD25)
- MEGA_CAMERA1 pad D26: (no net) -> Net-(MEGA_CAMERA1-PadD26)
- MEGA_CAMERA1 pad D27: (no net) -> Net-(MEGA_CAMERA1-PadD27)
- MEGA_CAMERA1 pad D28: (no net) -> Net-(MEGA_CAMERA1-PadD28)
- MEGA_CAMERA1 pad D29: (no net) -> Net-(MEGA_CAMERA1-PadD29)
- MEGA_CAMERA1 pad D3: /Camera/ENABLE_5V -> COIN_PIN
- MEGA_CAMERA1 pad D30: (no net) -> Net-(MEGA_CAMERA1-PadD30)
- MEGA_CAMERA1 pad D31: (no net) -> Net-(MEGA_CAMERA1-PadD31)
- MEGA_CAMERA1 pad D4: (no net) -> ENABLE_COIN_PIN
- MEGA_CAMERA1 pad D5: (no net) -> /Camera/ENABLE_5V
- MEGA_CAMERA1 pad D50: (no net) -> RADIO_MISO
- MEGA_CAMERA1 pad D51: (no net) -> RADIO_MOSI
- MEGA_CAMERA1 pad D52: (no net) -> RADIO_SCK
- MEGA_CAMERA1 pad D53: (no net) -> Net-(MEGA_CAMERA1-PadD53)
- MEGA_CAMERA1 pad D6: (no net) -> Net-(MEGA_CAMERA1-PadD6)
- MEGA_CAMERA1 pad D7: (no net) -> RADIO_CE
- MEGA_CAMERA1 pad D8: (no net) -> RADIO_CSN
- MEGA_CAMERA1 pad D9: (no net) -> ENABLE_MARQUEE
- MEGA_CAMERA1 pad MISO: (no net) -> Net-(MEGA_CAMERA1-PadMISO)
- MEGA_CAMERA1 pad MOSI: (no net) -> Net-(MEGA_CAMERA1-PadMOSI)
- MEGA_CAMERA1 pad RESET: (no net) -> Net-(MEGA_CAMERA1-PadRESET)
- MEGA_CAMERA1 pad RST: (no net) -> Net-(MEGA_CAMERA1-PadRST)
- MEGA_CAMERA1 pad RX: (no net) -> Net-(MEGA_CAMERA1-PadRX)
- MEGA_CAMERA1 pad SCK: (no net) -> Net-(MEGA_CAMERA1-PadSCK)
- MEGA_CAMERA1 pad TX: (no net) -> Net-(MEGA_CAMERA1-PadTX)
- MEGA_CAMERA1 pad VCC: (no net) -> Net-(MEGA_CAMERA1-PadVCC)
- MEGA_PAPER1 pad 5V: (no net) -> Net-(MEGA_PAPER1-Pad5V)
- MEGA_PAPER1 pad A0: (no net) -> Net-(MEGA_PAPER1-PadA0)
- MEGA_PAPER1 pad A1: (no net) -> Net-(MEGA_PAPER1-PadA1)
- MEGA_PAPER1 pad A10: (no net) -> Net-(MEGA_PAPER1-PadA10)
- MEGA_PAPER1 pad A11: (no net) -> Net-(MEGA_PAPER1-PadA11)
- MEGA_PAPER1 pad A12: (no net) -> Net-(MEGA_PAPER1-PadA12)
- MEGA_PAPER1 pad A13: (no net) -> Net-(MEGA_PAPER1-PadA13)
- MEGA_PAPER1 pad A14: (no net) -> Net-(MEGA_PAPER1-PadA14)
- MEGA_PAPER1 pad A15: (no net) -> Net-(MEGA_PAPER1-PadA15)
- MEGA_PAPER1 pad A2: (no net) -> Net-(MEGA_PAPER1-PadA2)
- MEGA_PAPER1 pad A3: (no net) -> Net-(MEGA_PAPER1-PadA3)
- MEGA_PAPER1 pad A4: (no net) -> Net-(MEGA_PAPER1-PadA4)
- MEGA_PAPER1 pad A5: (no net) -> Net-(MEGA_PAPER1-PadA5)
- MEGA_PAPER1 pad A6: (no net) -> Net-(MEGA_PAPER1-PadA6)
- MEGA_PAPER1 pad A7: (no net) -> Net-(MEGA_PAPER1-PadA7)
- MEGA_PAPER1 pad A8: (no net) -> Net-(MEGA_PAPER1-PadA8)
- MEGA_PAPER1 pad A9: (no net) -> Net-(MEGA_PAPER1-PadA9)
- MEGA_PAPER1 pad AREF: (no net) -> Net-(MEGA_PAPER1-PadAREF)
- MEGA_PAPER1 pad D10: (no net) -> Net-(MEGA_PAPER1-PadD10)
- MEGA_PAPER1 pad D11: (no net) -> Net-(MEGA_PAPER1-PadD11)
- MEGA_PAPER1 pad D12: (no net) -> Net-(MEGA_PAPER1-PadD12)
- MEGA_PAPER1 pad D13: (no net) -> Net-(MEGA_PAPER1-PadD13)
- MEGA_PAPER1 pad D14: (no net) -> /Camera/SERIAL_RX2
- MEGA_PAPER1 pad D15: (no net) -> /Paper/SERIAL_RX2
- MEGA_PAPER1 pad D16: (no net) -> Net-(MEGA_PAPER1-PadD16)
- MEGA_PAPER1 pad D17: (no net) -> Net-(MEGA_PAPER1-PadD17)
- MEGA_PAPER1 pad D18: (no net) -> Net-(MEGA_PAPER1-PadD18)
- MEGA_PAPER1 pad D19: (no net) -> Net-(MEGA_PAPER1-PadD19)
- MEGA_PAPER1 pad D2: (no net) -> /Camera/ORDER_INTERRUPT_PIN
- MEGA_PAPER1 pad D20: (no net) -> Net-(MEGA_PAPER1-PadD20)
- MEGA_PAPER1 pad D21: (no net) -> Net-(MEGA_PAPER1-PadD21)
- MEGA_PAPER1 pad D22: (no net) -> Net-(MEGA_PAPER1-PadD22)
- MEGA_PAPER1 pad D23: (no net) -> Net-(MEGA_PAPER1-PadD23)
- MEGA_PAPER1 pad D24: (no net) -> Net-(MEGA_PAPER1-PadD24)
- MEGA_PAPER1 pad D25: (no net) -> Net-(MEGA_PAPER1-PadD25)
- MEGA_PAPER1 pad D26: (no net) -> Net-(MEGA_PAPER1-PadD26)
- MEGA_PAPER1 pad D27: (no net) -> Net-(MEGA_PAPER1-PadD27)
- MEGA_PAPER1 pad D28: (no net) -> Net-(MEGA_PAPER1-PadD28)
- MEGA_PAPER1 pad D29: (no net) -> Net-(MEGA_PAPER1-PadD29)
- MEGA_PAPER1 pad D3: (no net) -> Net-(MEGA_PAPER1-PadD3)
- MEGA_PAPER1 pad D30: (no net) -> Net-(MEGA_PAPER1-PadD30)
- MEGA_PAPER1 pad D31: (no net) -> Net-(MEGA_PAPER1-PadD31)
- MEGA_PAPER1 pad D32: (no net) -> Net-(MEGA_PAPER1-PadD32)
- MEGA_PAPER1 pad D33: (no net) -> Net-(MEGA_PAPER1-PadD33)
- MEGA_PAPER1 pad D34: (no net) -> Net-(MEGA_PAPER1-PadD34)
- MEGA_PAPER1 pad D35: (no net) -> Net-(MEGA_PAPER1-PadD35)
- MEGA_PAPER1 pad D36: (no net) -> Net-(MEGA_PAPER1-PadD36)
- MEGA_PAPER1 pad D37: (no net) -> Net-(MEGA_PAPER1-PadD37)
- MEGA_PAPER1 pad D38: (no net) -> Net-(MEGA_PAPER1-PadD38)
- MEGA_PAPER1 pad D39: (no net) -> Net-(MEGA_PAPER1-PadD39)
- MEGA_PAPER1 pad D4: (no net) -> Net-(MEGA_PAPER1-PadD4)
- MEGA_PAPER1 pad D40: (no net) -> Net-(MEGA_PAPER1-PadD40)
- MEGA_PAPER1 pad D41: (no net) -> Net-(MEGA_PAPER1-PadD41)
- MEGA_PAPER1 pad D42: (no net) -> Net-(MEGA_PAPER1-PadD42)
- MEGA_PAPER1 pad D43: (no net) -> Net-(MEGA_PAPER1-PadD43)
- MEGA_PAPER1 pad D44: (no net) -> Net-(MEGA_PAPER1-PadD44)
- MEGA_PAPER1 pad D45: (no net) -> Net-(MEGA_PAPER1-PadD45)
- MEGA_PAPER1 pad D46: (no net) -> Net-(MEGA_PAPER1-PadD46)
- MEGA_PAPER1 pad D47: (no net) -> Net-(MEGA_PAPER1-PadD47)
- MEGA_PAPER1 pad D48: (no net) -> Net-(MEGA_PAPER1-PadD48)
- MEGA_PAPER1 pad D49: (no net) -> Net-(MEGA_PAPER1-PadD49)
- MEGA_PAPER1 pad D5: (no net) -> Net-(MEGA_PAPER1-PadD5)
- MEGA_PAPER1 pad D50: (no net) -> Net-(MEGA_PAPER1-PadD50)
- MEGA_PAPER1 pad D51: (no net) -> Net-(MEGA_PAPER1-PadD51)
- MEGA_PAPER1 pad D52: (no net) -> Net-(MEGA_PAPER1-PadD52)
- MEGA_PAPER1 pad D53: (no net) -> Net-(MEGA_PAPER1-PadD53)
- MEGA_PAPER1 pad D6: (no net) -> Net-(MEGA_PAPER1-PadD6)
- MEGA_PAPER1 pad D7: (no net) -> Net-(MEGA_PAPER1-PadD7)
- MEGA_PAPER1 pad D8: (no net) -> Net-(MEGA_PAPER1-PadD8)
- MEGA_PAPER1 pad D9: (no net) -> Net-(MEGA_PAPER1-PadD9)
- MEGA_PAPER1 pad MISO: (no net) -> Net-(MEGA_PAPER1-PadMISO)
- MEGA_PAPER1 pad MOSI: (no net) -> Net-(MEGA_PAPER1-PadMOSI)
- MEGA_PAPER1 pad RESET: (no net) -> Net-(MEGA_PAPER1-PadRESET)
- MEGA_PAPER1 pad RST: (no net) -> Net-(MEGA_PAPER1-PadRST)
- MEGA_PAPER1 pad RX: (no net) -> Net-(MEGA_PAPER1-PadRX)
- MEGA_PAPER1 pad SCK: (no net) -> Net-(MEGA_PAPER1-PadSCK)
- MEGA_PAPER1 pad TX: (no net) -> Net-(MEGA_PAPER1-PadTX)
- MEGA_PAPER1 pad VCC: (no net) -> Net-(MEGA_PAPER1-PadVCC)
- R_FLASH1 pad 2: (no net) -> FLASH_PIN
- R_FLASH2 pad 2: (no net) -> AUX_PIN
- U_MARQUEE1 pad 1: (no net) -> Net-(U_MARQUEE1-Pad1)
- U_MARQUEE1 pad 3: (no net) -> Net-(U_MARQUEE1-Pad3)
- U_MARQUEE1 pad 5: (no net) -> Net-(U_MARQUEE1-Pad5)
- U_MARQUEE1 pad 7: (no net) -> Net-(U_MARQUEE1-Pad7)
- U_RADIO1 pad 1: (no net) -> GND
- U_RADIO1 pad 2: (no net) -> 3V3_CAMERA
- U_RADIO1 pad 3: (no net) -> RADIO_CE
- U_RADIO1 pad 4: (no net) -> RADIO_CSN
- U_RADIO1 pad 5: (no net) -> RADIO_SCK
- U_RADIO1 pad 6: (no net) -> RADIO_MOSI
- U_RADIO1 pad 7: (no net) -> RADIO_MISO
- U_RADIO1 pad 8: (no net) -> RADIO_INTERRUPT
- U_STEP_DOWN_5V1 pad FB: (no net) -> Net-(U_STEP_DOWN_5V1-PadFB)
- U_STEP_DOWN_5V1 pad PG: (no net) -> Net-(U_STEP_DOWN_5V1-PadPG)
