File: hardware/kicad/nofilterbooth/nofilterbooth.sch (KiCad schematic (older format))
At the start: 2 parts

Commit message: clean
Parts:
- CONN_POWER_IN1: symbol Connector_Generic:Conn_01x02 -> nofilterbooth:Conn_01x02-Connector_Generic
- U_STEP_DOWN_5V1: symbol Converter_DCDC:D24V90F5 -> nofilterbooth:D24V90F5
Changed lines of the file:
@@
 $EndSheet
 $Comp
-L Connector_Generic:Conn_01x02 CONN_POWER_IN1
+L nofilterbooth:Conn_01x02-Connector_Generic CONN_POWER_IN1
 U 1 1 5E43D742
 P 4075 1075
@@
 $EndComp
 $Comp
-L power:+12V #PWR0123
+L nofilterbooth:+12V-power #PWR0123
 U 1 1 5E3BF560
 P 4075 1275
@@
 $EndComp
 $Comp
-L power:GND #PWR0124
+L nofilterbooth:GND-power #PWR0124
 U 1 1 5E3C03FE
 P 4175 1275
@@
 $EndComp
 $Comp
-L Converter_DCDC:D24V90F5 U_STEP_DOWN_5V1
+L nofilterbooth:D24V90F5 U_STEP_DOWN_5V1
 U 1 1 5E3C0E82
 P 6000 1125
@@
 $EndComp
 $Comp
-L power:+5V #PWR0128
+L nofilterbooth:+5V-power #PWR0128
 U 1 1 5E3C178D
 P 6200 1225
@@
 $EndComp
 $Comp
-L power:GND #PWR0126
+L nofilterbooth:GND-power #PWR0126
 U 1 1 5E3C0BAF
 P 6200 1425
@@
 $EndComp
 $Comp
-L power:GND #PWR0125
+L nofilterbooth:GND-power #PWR0125
 U 1 1 5E3BFE89
 P 5200 1425
@@
 $EndSheet
 $Comp
-L power:+12V #PWR0127
+L nofilterbooth:+12V-power #PWR0127
 U 1 1 5E3DD7DE
 P 5200 1225
