File: hardware/kicad/nofilterbooth/paper.sch (KiCad schematic (older format))
At the start: 1 part

Commit message: clean
Parts:
- MEGA_PAPER1: footprint MEGA2560PRO-EMBED:MEGA2560PRO-EMBED -> footprints:MEGA2560PRO-EMBED; symbol nofilterbooth-rescue:MEGA2560PRO-EMBED-MEGA2560PRO-EMBED-nofilterbooth-rescue -> nofilterbooth:MEGA2560PRO-EMBED
Changed lines of the file:
@@
 $EndDescr
 $Comp
-L nofilterbooth-rescue:MEGA2560PRO-EMBED-MEGA2560PRO-EMBED-nofilterbooth-rescue MEGA_PAPER?
+L nofilterbooth:MEGA2560PRO-EMBED MEGA_PAPER?
 U 1 1 5E40A8A4
 P 3150 3400
@@
 F 0 "MEGA_PAPER1" H 3150 5567 50  0000 C CNN
 F 1 "MEGA2560PRO-EMBED" H 3150 5476 50  0000 C CNN
-F 2 "MEGA2560PRO-EMBED:MEGA2560PRO-EMBED" V 3100 2000 50  0001 L BNN
+F 2 "footprints:MEGA2560PRO-EMBED" V 3100 2000 50  0001 L BNN
 F 3 "" H 3150 3400 50  0001 C CNN
 	1    3150 3400
