File: hardware/kicad/camera.sch (KiCad schematic (older format))
At the start: 62 parts

Commit message: kicad schematic & pcb v0.1
Parts:
- added C_CAMERA_5V1, C_RTC1: 100nF, Capacitor_THT:C_Disc_D3.0mm_W1.6mm_P2.50mm, symbol 1nofilterbooth:C-Device
- added C_LORA1: 100uF, Capacitor_THT:CP_Radial_D10.0mm_P5.00mm, symbol 1nofilterbooth:CP-Device
- added R_RXD_LORA1, R_TXD_LORA1: 4.7k 1/2W, Resistor_THT:R_Axial_DIN0309_L9.0mm_D3.2mm_P12.70mm_Horizontal, symbol 1nofilterbooth:R_Small-Device
- added URTC1: RTC_DS3231_BREAKOUT, 1nofilterbooth:DS3231_breakout, symbol 1nofilterbooth:RTC_DS3231_BREAKOUT
- added U_RADIO_LORA1: SX17278_LORA, 1nofilterbooth:LORA_E32-TTL-100, symbol 1nofilterbooth:SX17278_LORA
- CONN_AUX1, CONN_FLASH1: value Conn_01x02 -> XT60; symbol nofilterbooth:Conn_01x02-Connector_Generic -> 1nofilterbooth:Conn_01x02-Connector_Generic
- CONN_BATT1, CONN_SW_SCISSOR1, CONN_SW_SHUTTER1: symbol nofilterbooth:Conn_01x02-Connector_Generic -> 1nofilterbooth:Conn_01x02-Connector_Generic
- CONN_CEILING1, CONN_MARQUEE_WS2811, CONN_SW_PAP1, CONN_SW_PAP2, CONN_SW_PAP3, CONN_SW_PAP4: symbol nofilterbooth:Conn_01x03-Connector_Generic -> 1nofilterbooth:Conn_01x03-Connector_Generic
- CONN_COIN1, CONN_LUXSENSOR1, CONN_SEGMENT1, CONN_START1, CONN_STEP_PAPER1, CONN_STEP_SCISSOR1, CONN_STEP_SHUTTER1: symbol nofilterbooth:Conn_01x04-Connector_Generic -> 1nofilterbooth:Conn_01x04-Connector_Generic
- CONN_MATRIX1: symbol nofilterbooth:Conn_01x05-Connector_Generic -> 1nofilterbooth:Conn_01x05-Connector_Generic
- C_ATTINY1, C_AUX1, C_CEILING1, C_FLASH1, C_START1: symbol nofilterbooth:CP-Device -> 1nofilterbooth:CP-Device
- C_COIN1, C_LUXSENSOR1, C_SEGMENT1: footprint (none) -> Capacitor_THT:C_Disc_D3.0mm_W1.6mm_P2.50mm; symbol nofilterbooth:C-Device -> 1nofilterbooth:C-Device
- C_DRV_PAPER1: renamed from C1; symbol nofilterbooth:CP-Device -> 1nofilterbooth:CP-Device
- C_DRV_SCISSOR1: renamed from C3; symbol nofilterbooth:CP-Device -> 1nofilterbooth:CP-Device
- C_DRV_SHUTTER1: renamed from C2; symbol nofilterbooth:CP-Device -> 1nofilterbooth:CP-Device
- C_MARQUEE1: renamed from C_AUX2; symbol nofilterbooth:CP-Device -> 1nofilterbooth:CP-Device
- C_MATRIX1: symbol nofilterbooth:C-Device -> 1nofilterbooth:C-Device
- C_RADIO1: value 10uF -> 470uF; symbol nofilterbooth:CP-Device -> 1nofilterbooth:CP-Device
- DRV_PAPER1, DRV_SCISSOR1, DRV_SHUTTER1: symbol nofilterbooth:Pololu_Breakout_DRV8825 -> 1nofilterbooth:Pololu_Breakout_DRV8825
- LED_SW_PAPER1, LED_SW_PAPER2, LED_SW_PAPER3, LED_SW_PAPER4: symbol nofilterbooth:LED_Small-Device -> 1nofilterbooth:LED_Small-Device
- LED_SW_SCISSOR1, LED_SW_SHUTTER1, LED_SW_START1: value LED_Small -> LED 3mm; symbol nofilterbooth:LED_Small-Device -> 1nofilterbooth:LED_Small-Device
- MEGA_CAMERA1: footprint footprints:MEGA2560PRO-EMBED -> 1nofilterbooth:MEGA2560PRO-EMBED; symbol nofilterbooth:MEGA2560PRO-EMBED -> 1nofilterbooth:MEGA2560PRO-EMBED
- Q_AUX1, Q_FLASH1, Q_START1: symbol nofilterbooth:TIP120-Transistor_BJT -> 1nofilterbooth:TIP120-Transistor_BJT
- R_BATT1, R_BATT2, R_FLASH1, R_FLASH2, R_MARQUEE1, R_START1, R_SW_PAPER1, R_SW_PAPER2, R_SW_PAPER3, R_SW_PAPER4, R_SW_SCISSOR1, R_SW_SHUTTER1, R_SW_START1: symbol nofilterbooth:R_Small-Device -> 1nofilterbooth:R_Small-Device
- U_MARQUEE1: symbol nofilterbooth:ATtiny85-20PU-MCU_Microchip_ATtiny -> 1nofilterbooth:ATtiny85-20PU-MCU_Microchip_ATtiny
- U_RADIO1: symbol nofilterbooth:NRF24L01_Breakout-RF -> 1nofilterbooth:NRF24L01_Breakout-RF
Connections:
- net labels added: LORA_AUX, LORA_M0, LORA_M1, LORA_RXD, LORA_TXD
- net labels removed: +12V-power, +5V-power, GND-power
- wire segments 118 -> 143

Commit message: correction schematic gilou
Parts:
- C_ATTINY1: footprint Capacitor_THT:CP_Radial_D10.0mm_P5.00mm -> Capacitor_THT:C_Rect_L7.2mm_W2.5mm_P5.00mm_FKS2_FKP2_MKS2_MKP2
- C_CAMERA_5V1, C_COIN1, C_LUXSENSOR1, C_MATRIX1, C_RTC1, C_SEGMENT1: footprint Capacitor_THT:C_Disc_D3.0mm_W1.6mm_P2.50mm -> Capacitor_THT:C_Rect_L7.2mm_W2.5mm_P5.00mm_FKS2_FKP2_MKS2_MKP2
- C_MARQUEE1: value 1000uF 16v -> 1000uF
- R_BATT1, R_BATT2, R_FLASH1, R_FLASH2, R_MARQUEE1, R_RXD_LORA1, R_START1, R_SW_PAPER1, R_SW_PAPER2, R_SW_PAPER3, R_SW_PAPER4, R_SW_SCISSOR1, R_SW_SHUTTER1, R_SW_START1, R_TXD_LORA1: footprint Resistor_THT:R_Axial_DIN0309_L9.0mm_D3.2mm_P12.70mm_Horizontal -> Resistor_THT:R_Axial_DIN0207_L6.3mm_D2.5mm_P10.16mm_Horizontal
Connections:
- net 3V3_CAMERA renamed +3V3
- net 5V_CAMERA renamed +5C
- no-connect marks 9 -> 35
Other:
- moved on the sheet: C_ATTINY1, C_RTC1, URTC1

Commit message: update, gilou dans la place
Parts:
- removed C_RADIO1: 470uF, Capacitor_THT:CP_Radial_D10.0mm_P5.00mm, symbol 1nofilterbooth:CP-Device
- removed C_START1: 100uF, Capacitor_THT:CP_Radial_D10.0mm_P5.00mm, symbol 1nofilterbooth:CP-Device
- removed Q_START1: TIP120, Package_TO_SOT_THT:TO-220-3_Vertical, symbol 1nofilterbooth:TIP120-Transistor_BJT
- added CONN_COUNT1: WIRE, Connector_PinHeader_2.54mm:PinHeader_1x02_P2.54mm_Vertical, symbol 1nofilterbooth:Conn_01x02-Connector_Generic
- added C_CAMERA_5V2: 100nF, Capacitor_THT:C_Rect_L7.2mm_W2.5mm_P5.00mm_FKS2_FKP2_MKS2_MKP2, symbol 1nofilterbooth:C-Device
- added Q_COUNT1, Q_COUNT2: BC327, Package_TO_SOT_THT:TO-92L_HandSolder, symbol Device:Q_NPN_CBE
- added R_FLASH3: 2.2k 1/2W, Resistor_THT:R_Axial_DIN0207_L6.3mm_D2.5mm_P10.16mm_Horizontal, symbol 1nofilterbooth:R_Small-Device
- added R_SW_PAPER5: 560ohm 1/2W, Resistor_THT:R_Axial_DIN0207_L6.3mm_D2.5mm_P10.16mm_Horizontal, symbol 1nofilterbooth:R_Small-Device
- CONN_BATT1, CONN_SW_SCISSOR1, CONN_SW_SHUTTER1: footprint Connector_JST:JST_XH_S2B-XH-A_1x02_P2.50mm_Horizontal -> Connector_JST:JST_XH_S2B-XH-A-1_1x02_P2.50mm_Horizontal
- CONN_CEILING1, CONN_MARQUEE_WS2811, CONN_SW_PAP1, CONN_SW_PAP2, CONN_SW_PAP3, CONN_SW_PAP4: footprint Connector_JST:JST_XH_S3B-XH-A_1x03_P2.50mm_Horizontal -> Connector_JST:JST_XH_S3B-XH-A-1_1x03_P2.50mm_Horizontal
- CONN_COIN1, CONN_LUXSENSOR1, CONN_SEGMENT1, CONN_START1, CONN_STEP_PAPER1, CONN_STEP_SCISSOR1, CONN_STEP_SHUTTER1: value Conn_01x04 -> JST_XH4; footprint Connector_JST:JST_XH_S4B-XH-A_1x04_P2.50mm_Horizontal -> Connector_JST:JST_XH_S4B-XH-A-1_1x04_P2.50mm_Horizontal
- CONN_MATRIX1: value Conn_01x05 -> JST_XH5; footprint Connector_JST:JST_XH_S5B-XH-A_1x05_P2.50mm_Horizontal -> Connector_JST:JST_XH_S5B-XH-A-1_1x05_P2.50mm_Horizontal
- C_ATTINY1: value 0.1uF -> 100nF
- C_AUX1, C_FLASH1: value 100uF -> 680uF; footprint Capacitor_THT:CP_Radial_D10.0mm_P5.00mm -> Capacitor_THT:CP_Radial_D8.0mm_P3.50mm
- C_CEILING1, C_DRV_PAPER1, C_DRV_SCISSOR1, C_DRV_SHUTTER1, C_LORA1: footprint Capacitor_THT:CP_Radial_D10.0mm_P5.00mm -> Capacitor_THT:CP_Radial_D6.3mm_P2.50mm
- C_MARQUEE1: value 1000uF -> 680uF; footprint Capacitor_THT:CP_Radial_D10.0mm_P5.00mm -> Capacitor_THT:CP_Radial_D8.0mm_P3.50mm
Connections:
- net +12V: now also CONN_COUNT1.1 (Pin_1), C_CAMERA_5V2.1
- net AUX_PIN: now also MEGA_CAMERA1.D46; no longer MEGA_CAMERA1.D26
- net ENABLE_5V: now also MEGA_CAMERA1.D44; no longer MEGA_CAMERA1.D29
- net FLASH_PIN: now also MEGA_CAMERA1.D45; no longer MEGA_CAMERA1.D27
- net GND: now also C_CAMERA_5V2.2, Q_COUNT1.3 (E), Q_COUNT2.3 (E)
- net PAPER_M0: now also MEGA_CAMERA1.D35; no longer MEGA_CAMERA1.D33
- net PAPER_PIN_DIR: now also MEGA_CAMERA1.D34; no longer MEGA_CAMERA1.D35
- net PAPER_PIN_STP: now also MEGA_CAMERA1.D33; no longer MEGA_CAMERA1.D34
- net PAPER_SWITCH1_PIN: now also MEGA_CAMERA1.D30; no longer MEGA_CAMERA1.D46
- net PAPER_SWITCH2_PIN: now also MEGA_CAMERA1.D31; no longer MEGA_CAMERA1.D47
- net PAPER_SWITCH3_PIN: now also MEGA_CAMERA1.D28; no longer MEGA_CAMERA1.D48
- net PAPER_SWITCH4_PIN: now also MEGA_CAMERA1.D29; no longer MEGA_CAMERA1.D49
- net RADIO_CE: now also MEGA_CAMERA1.D48; no longer MEGA_CAMERA1.D7
- net RADIO_CSN: now also MEGA_CAMERA1.D49; no longer MEGA_CAMERA1.D8
- net SCISSOR_ENDSTOP_PIN: now also MEGA_CAMERA1.D27; no longer MEGA_CAMERA1.D45
- net SCISSOR_M0: now also MEGA_CAMERA1.D43; no longer MEGA_CAMERA1.D41
- net SCISSOR_PIN_DIR: now also MEGA_CAMERA1.D41; no longer MEGA_CAMERA1.D39
- net SCISSOR_PIN_ENABLE: now also MEGA_CAMERA1.D42; no longer MEGA_CAMERA1.D40
- net SCISSOR_PIN_STP: now also MEGA_CAMERA1.D40; no longer MEGA_CAMERA1.D38
- net SHUTTER_ENDSTOP_PIN: now also MEGA_CAMERA1.D26; no longer MEGA_CAMERA1.D44
- net SHUTTER_M0: now also MEGA_CAMERA1.D36; no longer MEGA_CAMERA1.D37
- net SHUTTER_PIN_DIR: now also MEGA_CAMERA1.D38; no longer MEGA_CAMERA1.D43
- net SHUTTER_PIN_ENABLE: now also MEGA_CAMERA1.D39; no longer MEGA_CAMERA1.D36
- net SHUTTER_PIN_STP: now also MEGA_CAMERA1.D37; no longer MEGA_CAMERA1.D42
- net at CONN_START1.4 (Pin_4): now also R_SW_PAPER5.1
- net at R_START1.1: now also Q_COUNT2.2 (B)
- new net: CONN_COUNT1.2 (Pin_2), Q_COUNT1.1 (C)
- new net: Q_COUNT1.2 (B), R_FLASH3.1
- new net: Q_COUNT2.1 (C), R_SW_PAPER5.2
- new net COUNT_PIN: MEGA_CAMERA1.D8, R_FLASH3.2
- no-connect marks 35 -> 34
Other:
- moved on the sheet: C_RTC1, URTC1

Commit message: pcb finalized
Parts:
- removed R_SW_PAPER5: 560ohm 1/2W, Resistor_THT:R_Axial_DIN0207_L6.3mm_D2.5mm_P10.16mm_Horizontal, symbol 1nofilterbooth:R_Small-Device
- added J_AUX_CAM1: Conn_01x10, Connector_PinHeader_2.54mm:PinHeader_1x05_P2.54mm_Vertical, symbol Connector_Generic:Conn_01x05
- added R_LED_START1: 560ohm, Resistor_THT:R_Axial_DIN0207_L6.3mm_D2.5mm_P10.16mm_Horizontal, symbol 1nofilterbooth:R_Small-Device
- R_BATT1: value 20k1/2W -> 20k
- R_BATT2: value 10k 1/2W -> 10k
- R_FLASH1, R_FLASH2, R_FLASH3, R_START1: value 2.2k 1/2W -> 2.2k
- R_MARQUEE1: value 430ohm 1/2W -> 430ohm
- R_RXD_LORA1, R_TXD_LORA1: value 4.7k 1/2W -> 4.7k
- R_SW_PAPER1, R_SW_PAPER2, R_SW_PAPER3, R_SW_PAPER4, R_SW_SCISSOR1, R_SW_SHUTTER1, R_SW_START1: value 560ohm 1/2W -> 560ohm
- U_MARQUEE1: value ATtiny85-20PU -> ATtiny85
- renumbered Q_COUNT2 to Q_START1
Connections:
- net A13: now reaches MEGA_CAMERA1.A13
- net A13: now also J_AUX_CAM1.5 (Pin_5)
- net A14: now reaches MEGA_CAMERA1.A14
- net A14: now also J_AUX_CAM1.4 (Pin_4)
- net D47: now reaches MEGA_CAMERA1.D47
- net D47: now also J_AUX_CAM1.3 (Pin_3)
- net D53: now reaches MEGA_CAMERA1.D53
- net D53: now also J_AUX_CAM1.2 (Pin_2)
- net D7: now reaches MEGA_CAMERA1.D7
- net D7: now also J_AUX_CAM1.1 (Pin_1)
- net at CONN_START1.4 (Pin_4): now also R_LED_START1.1
- net at Q_START1.1 (C): now also R_LED_START1.2
- no-connect marks 34 -> 29
Changed lines of the file:
@@
 P 14275 1000
 F 0 "R_SW_SHUTTER1" V 14079 1000 50  0000 C CNN
-F 1 "560ohm 1/2W" V 14170 1000 50  0000 C CNN
+F 1 "560ohm" V 14170 1000 50  0000 C CNN
 F 2 "Resistor_THT:R_Axial_DIN0207_L6.3mm_D2.5mm_P10.16mm_Horizontal" H 14275 1000 50  0001 C CNN
 F 3 "~" H 14275 1000 50  0001 C CNN
@@
 P 14275 1900
 F 0 "R_SW_SCISSOR1" V 14079 1900 50  0000 C CNN
-F 1 "560ohm 1/2W" V 14170 1900 50  0000 C CNN
+F 1 "560ohm" V 14170 1900 50  0000 C CNN
 F 2 "Resistor_THT:R_Axial_DIN0207_L6.3mm_D2.5mm_P10.16mm_Horizontal" H 14275 1900 50  0001 C CNN
 F 3 "~" H 14275 1900 50  0001 C CNN
@@
 P 14075 3500
 F 0 "R_SW_PAPER2" V 13879 3500 50  0000 C CNN
-F 1 "560ohm 1/2W" V 13970 3500 50  0000 C CNN
+F 1 "560ohm" V 13970 3500 50  0000 C CNN
 F 2 "Resistor_THT:R_Axial_DIN0207_L6.3mm_D2.5mm_P10.16mm_Horizontal" H 14075 3500 50  0001 C CNN
 F 3 "~" H 14075 3500 50  0001 C CNN
@@
 P 14075 4300
 F 0 "R_SW_PAPER3" V 13879 4300 50  0000 C CNN
-F 1 "560ohm 1/2W" V 13970 4300 50  0000 C CNN
+F 1 "560ohm" V 13970 4300 50  0000 C CNN
 F 2 "Resistor_THT:R_Axial_DIN0207_L6.3mm_D2.5mm_P10.16mm_Horizontal" H 14075 4300 50  0001 C CNN
 F 3 "~" H 14075 4300 50  0001 C CNN
@@
 P 14075 5000
 F 0 "R_SW_PAPER4" V 13879 5000 50  0000 C CNN
-F 1 "560ohm 1/2W" V 13970 5000 50  0000 C CNN
+F 1 "560ohm" V 13970 5000 50  0000 C CNN
 F 2 "Resistor_THT:R_Axial_DIN0207_L6.3mm_D2.5mm_P10.16mm_Horizontal" H 14075 5000 50  0001 C CNN
 F 3 "~" H 14075 5000 50  0001 C CNN
@@
 P 4250 1175
 F 0 "R_FLASH1" V 4054 1175 50  0000 C CNN
-F 1 "2.2k 1/2W" V 4145 1175 50  0000 C CNN
+F 1 "2.2k" V 4145 1175 50  0000 C CNN
 F 2 "Resistor_THT:R_Axial_DIN0207_L6.3mm_D2.5mm_P10.16mm_Horizontal" H 4250 1175 50  0001 C CNN
 F 3 "~" H 4250 1175 50  0001 C CNN
@@
 P 6450 1150
 F 0 "R_FLASH2" V 6254 1150 50  0000 C CNN
-F 1 "2.2k 1/2W" V 6345 1150 50  0000 C CNN
+F 1 "2.2k" V 6345 1150 50  0000 C CNN
 F 2 "Resistor_THT:R_Axial_DIN0207_L6.3mm_D2.5mm_P10.16mm_Horizontal" H 6450 1150 50  0001 C CNN
 F 3 "~" H 6450 1150 50  0001 C CNN
@@
 P 9200 1475
 F 0 "U_MARQUEE1" H 9800 900 50  0000 R CNN
-F 1 "ATtiny85-20PU" H 9900 825 50  0000 R CNN
+F 1 "ATtiny85" H 9900 825 50  0000 R CNN
 F 2 "Package_DIP:DIP-8_W7.62mm" H 9200 1475 50  0001 C CIN
 F 3 "http://ww1.microchip.com/downloads/en/DeviceDoc/atmel-2586-avr-8-bit-microcontroller-attiny25-attiny45-attiny85_datasheet.pdf" H 9200 1475 50  0001 C CNN
@@
 P 8800 3575
 F 0 "R_BATT1" H 9025 3625 50  0000 C CNN
-F 1 "20k1/2W" H 9050 3550 50  0000 C CNN
+F 1 "20k" H 9050 3550 50  0000 C CNN
 F 2 "Resistor_THT:R_Axial_DIN0207_L6.3mm_D2.5mm_P10.16mm_Horizontal" H 8800 3575 50  0001 C CNN
 F 3 "~" H 8800 3575 50  0001 C CNN
@@
 P 8800 4125
 F 0 "R_BATT2" H 9025 4175 50  0000 C CNN
-F 1 "10k 1/2W" H 9050 4100 50  0000 C CNN
+F 1 "10k" H 9050 4100 50  0000 C CNN
 F 2 "Resistor_THT:R_Axial_DIN0207_L6.3mm_D2.5mm_P10.16mm_Horizontal" H 8800 4125 50  0001 C CNN
 F 3 "~" H 8800 4125 50  0001 C CNN
@@
 P 10100 1275
 F 0 "R_MARQUEE1" V 10025 1250 50  0000 C CNN
-F 1 "430ohm 1/2W" V 10175 1250 50  0000 C CNN
+F 1 "430ohm" V 10175 1250 50  0000 C CNN
 F 2 "Resistor_THT:R_Axial_DIN0207_L6.3mm_D2.5mm_P10.16mm_Horizontal" H 10100 1275 50  0001 C CNN
 F 3 "~" H 10100 1275 50  0001 C CNN
@@
 	1    0    0    -1
 $EndComp
-Wire Wire Line
-	13650 7275 13575 7275
 $Comp
 L 1nofilterbooth:+12V-power #PWR0158
@@
 P 13175 7075
 F 0 "R_START1" V 12979 7075 50  0000 C CNN
-F 1 "2.2k 1/2W" V 13070 7075 50  0000 C CNN
+F 1 "2.2k" V 13070 7075 50  0000 C CNN
 F 2 "Resistor_THT:R_Axial_DIN0207_L6.3mm_D2.5mm_P10.16mm_Horizontal" H 13175 7075 50  0001 C CNN
 F 3 "~" H 13175 7075 50  0001 C CNN
@@
 Wire Wire Line
 	13725 6875 13725 6950
-Wire Wire Line
-	13725 6950 13900 6950
 Text Notes 14750 6975 0    50   ~ 0
 To GND start bulb
@@
 P 13575 6550
 F 0 "R_SW_START1" V 13379 6550 50  0000 C CNN
-F 1 "560ohm 1/2W" V 13470 6550 50  0000 C CNN
+F 1 "560ohm" V 13470 6550 50  0000 C CNN
 F 2 "Resistor_THT:R_Axial_DIN0207_L6.3mm_D2.5mm_P10.16mm_Horizontal" H 13575 6550 50  0001 C CNN
 F 3 "~" H 13575 6550 50  0001 C CNN
@@
 P 14075 2700
 F 0 "R_SW_PAPER1" V 13879 2700 50  0000 C CNN
-F 1 "560ohm 1/2W" V 13970 2700 50  0000 C CNN
+F 1 "560ohm" V 13970 2700 50  0000 C CNN
 F 2 "Resistor_THT:R_Axial_DIN0207_L6.3mm_D2.5mm_P10.16mm_Horizontal" H 14075 2700 50  0001 C CNN
 F 3 "~" H 14075 2700 50  0001 C CNN
@@
 P 7275 7225
 F 0 "R_RXD_LORA1" V 7079 7225 50  0000 C CNN
-F 1 "4.7k 1/2W" V 7170 7225 50  0000 C CNN
+F 1 "4.7k" V 7170 7225 50  0000 C CNN
 F 2 "Resistor_THT:R_Axial_DIN0207_L6.3mm_D2.5mm_P10.16mm_Horizontal" H 7275 7225 50  0001 C CNN
 F 3 "" H 7275 7225 50  0001 C CNN
@@
 P 7275 7525
 F 0 "R_TXD_LORA1" V 7079 7525 50  0000 C CNN
-F 1 "4.7k 1/2W" V 7170 7525 50  0000 C CNN
+F 1 "4.7k" V 7170 7525 50  0000 C CNN
 F 2 "Resistor_THT:R_Axial_DIN0207_L6.3mm_D2.5mm_P10.16mm_Horizontal" H 7275 7525 50  0001 C CNN
 F 3 "" H 7275 7525 50  0001 C CNN
@@
 NoConn ~ 5925 4475
 NoConn ~ 5925 4575
-NoConn ~ 5925 4675
-NoConn ~ 5925 4775
-NoConn ~ 5925 7075
 $Comp
 L power:GND #PWR0208
@@
 Text Label 4925 6975 2    50   ~ 0
 PAPER_SWITCH4_PIN
-NoConn ~ 5925 6475
 NoConn ~ 4925 7375
-NoConn ~ 4925 4775
 $Comp
 L 1nofilterbooth:Conn_01x02-Connector_Generic CONN_AUX?
@@
 P 6425 2575
 F 0 "R_FLASH3" V 6229 2575 50  0000 C CNN
-F 1 "2.2k 1/2W" V 6320 2575 50  0000 C CNN
+F 1 "2.2k" V 6320 2575 50  0000 C CNN
 F 2 "Resistor_THT:R_Axial_DIN0207_L6.3mm_D2.5mm_P10.16mm_Horizontal" H 6425 2575 50  0001 C CNN
 F 3 "~" H 6425 2575 50  0001 C CNN
@@
 COUNT_PIN
 $Comp
-L Device:Q_NPN_CBE Q_COUNT2
+L Device:Q_NPN_CBE Q_START1
 U 1 1 5E4EAB32
 P 13475 7075
-F 0 "Q_COUNT2" H 13666 7121 50  0000 L CNN
+F 0 "Q_START1" H 13666 7121 50  0000 L CNN
 F 1 "BC327" H 13666 7030 50  0000 L CNN
 F 2 "Package_TO_SOT_THT:TO-92L_HandSolder" H 13675 7175 50  0001 C CNN
@@
 	1    0    0    -1
 $EndComp
-Connection ~ 13575 7275
 Wire Wire Line
 	14250 6650 14475 6650
@@
 Connection ~ 6825 2775
 $Comp
-L 1nofilterbooth:R_Small-Device R_SW_PAPER5
-U 1 1 5E60AC52
-P 14000 6950
-F 0 "R_SW_PAPER5" V 13804 6950 50  0000 C CNN
-F 1 "560ohm 1/2W" V 13895 6950 50  0000 C CNN
-F 2 "Resistor_THT:R_Axial_DIN0207_L6.3mm_D2.5mm_P10.16mm_Horizontal" H 14000 6950 50  0001 C CNN
-F 3 "~" H 14000 6950 50  0001 C CNN
-	1    14000 6950
-	0    1    1    0
-$EndComp
-Wire Wire Line
-	14100 6950 14475 6950
+L Connector_Generic:Conn_01x05 J_AUX_CAM1
+U 1 1 5E5138FB
+P 1500 8900
+F 0 "J_AUX_CAM1" H 1418 8475 50  0000 C CNN
+F 1 "Conn_01x10" H 1418 8566 50  0000 C CNN
+F 2 "Connector_PinHeader_2.54mm:PinHeader_1x05_P2.54mm_Vertical" H 1500 8900 50  0001 C CNN
+F 3 "~" H 1500 8900 50  0001 C CNN
+	1    1500 8900
+	-1   0    0    1
+$EndComp
+Text Label 1700 9100 0    50   ~ 0
+D7
+Text Label 4925 4775 2    50   ~ 0
+D7
+Text Label 5925 7075 0    50   ~ 0
+D53
+Text Label 5925 6475 0    50   ~ 0
+D47
+Text Label 5925 4775 0    50   ~ 0
+A14
+Text Label 5925 4675 0    50   ~ 0
+A13
+Text Label 1700 9000 0    50   ~ 0
+D53
+Text Label 1700 8900 0    50   ~ 0
+D47
+Text Label 1700 8800 0    50   ~ 0
+A14
+Text Label 1700 8700 0    50   ~ 0
+A13
+Wire Wire Line
+	13725 6950 14000 6950
+$Comp
+L 1nofilterbooth:R_Small-Device R_LED_START1
+U 1 1 5E4ACE71
+P 14100 6950
+F 0 "R_LED_START1" V 13904 6950 50  0000 C CNN
+F 1 "560ohm" V 13995 6950 50  0000 C CNN
+F 2 "Resistor_THT:R_Axial_DIN0207_L6.3mm_D2.5mm_P10.16mm_Horizontal" H 14100 6950 50  0001 C CNN
+F 3 "~" H 14100 6950 50  0001 C CNN
+	1    14100 6950
+	0    1    1    0
+$EndComp
+Wire Wire Line
+	14200 6950 14475 6950
 $EndSCHEMATC
