File: hardware/kicad/nofilterbooth.kicad_pcb (KiCad board)
At the start: 2 copper layers, 101 parts

Commit message: correction schematic gilou
Parts:
- added H1: MountingHole, MountingHole:MountingHole_3.2mm_M3, F.Cu at (140.2, 140.4)
- added H2: MountingHole, MountingHole:MountingHole_3.2mm_M3, F.Cu at (140.2, 148.3)
- added H3: MountingHole, MountingHole:MountingHole_3.2mm_M3, F.Cu at (148.2, 140.4)
- added H4: MountingHole, MountingHole:MountingHole_3.2mm_M3, F.Cu at (148.2, 148.3)
- added H5: MountingHole, MountingHole:MountingHole_3.2mm_M3, F.Cu at (156.1, 140.4)
- added H6: MountingHole, MountingHole:MountingHole_3.2mm_M3, F.Cu at (156.1, 148.3)
- added H7: MountingHole, MountingHole:MountingHole_3.2mm_M3, F.Cu at (164.1, 140.4)
- added H8: MountingHole, MountingHole:MountingHole_3.2mm_M3, F.Cu at (164.1, 148.3)
- C_ATTINY1: footprint Capacitor_THT:CP_Radial_D10.0mm_P5.00mm -> Capacitor_THT:C_Rect_L7.2mm_W2.5mm_P5.00mm_FKS2_FKP2_MKS2_MKP2
- C_CAMERA_5V1, C_COIN1, C_LUXSENSOR1, C_MATRIX1, C_MEGA_PAPER1, C_RTC1, C_SEGMENT1: footprint Capacitor_THT:C_Disc_D3.0mm_W1.6mm_P2.50mm -> Capacitor_THT:C_Rect_L7.2mm_W2.5mm_P5.00mm_FKS2_FKP2_MKS2_MKP2
- C_MARQUEE1: value 1000uF 16v -> 1000uF
- R_BATT1, R_BATT2, R_FLASH1, R_FLASH2, R_MARQUEE1, R_RXD_LORA1, R_START1, R_SW_BOTTOM1, R_SW_MIDDLE1, R_SW_PAPER1, R_SW_PAPER2, R_SW_PAPER3, R_SW_PAPER4, R_SW_ROT1, R_SW_ROT2, R_SW_SCISSOR1, R_SW_SHUTTER1, R_SW_START1, R_SW_UP1, R_TXD_LORA1: footprint Resistor_THT:R_Axial_DIN0309_L9.0mm_D3.2mm_P12.70mm_Horizontal -> Resistor_THT:R_Axial_DIN0207_L6.3mm_D2.5mm_P10.16mm_Horizontal
- moved CONN_FLASH1 1.42 mm to (130.2, 119.4)
- moved C_DRV_SCISSOR1 1.42 mm to (280.0, 113.0)
- moved R_FLASH2 1.42 mm to (140.3, 83.8)
- moved C_LUXSENSOR1 1.42 mm to (225.4, 34.3)
- moved C_RADIO1 1.42 mm to (175.9, 52.1)
- moved Q_START1 1.42 mm to (203.8, 41.9)
- moved R_FLASH1 1.42 mm to (127.6, 83.8)
- moved CONN_START1 1.42 mm to (211.5, 27.9)
- moved CONN_STEP_SHUTTER1 1.42 mm to (235.6, 114.3)
- moved C_AUX1 1.42 mm to (140.3, 94.0)
- moved C_DRV_SHUTTER1 1.42 mm to (249.6, 113.0)
- moved DRV_PAPER1 1.42 mm to (217.8, 104.1)
- moved Q_AUX1 1.42 mm to (140.3, 104.1)
- moved R_BATT1 1.42 mm to (158.1, 108.0)
- moved R_RXD_LORA1 1.42 mm to (200.0, 88.9)
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Connections:
- net 3V3_CAMERA renamed +3V3
- C_ATTINY1 pad 1: 5V_CAMERA -> +5C
- MEGA_CAMERA1 pad 5V: 5V_CAMERA -> +5C
- MEGA_PAPER1 pad 5V: (no net) -> +5C
- U_MARQUEE1 pad 8: 5V_CAMERA -> +5C
- U_STEP_DOWN_5V1 pad VOUT: Net-(U_STEP_DOWN_5V1-PadVOUT) -> +5V
Routing:
- added copper zone on B.Cu, net GND
Other:
- board outline added: 270 x 90 mm

Commit message: update, gilou dans la place
Parts:
- removed C_RADIO1: 470uF, Capacitor_THT:CP_Radial_D10.0mm_P5.00mm
- removed C_START1: 100uF, Capacitor_THT:CP_Radial_D10.0mm_P5.00mm
- removed H5, H6, H7, H8: MountingHole, MountingHole:MountingHole_3.2mm_M3
- removed Q_START1: TIP120, Package_TO_SOT_THT:TO-220-3_Vertical
- added CONN_COUNT1: WIRE, Connector_PinHeader_2.54mm:PinHeader_1x02_P2.54mm_Vertical, F.Cu at (270.5, 40.6)
- added CONN_FAN1: JST_XH2, Connector_JST:JST_XH_S2B-XH-A-1_1x02_P2.50mm_Horizontal, F.Cu at (78.7, 113.8)
- added C_AUX3: 680uF, Capacitor_THT:CP_Radial_D8.0mm_P3.50mm, F.Cu at (77.5, 90.2)
- added C_CAMERA_5V2: 100nF, Capacitor_THT:C_Rect_L7.2mm_W2.5mm_P5.00mm_FKS2_FKP2_MKS2_MKP2, F.Cu at (270.5, 44.5)
- added Q_AUX2: TIP120, Package_TO_SOT_THT:TO-220-3_Vertical, F.Cu at (72.4, 101.6)
- added Q_COUNT1: BC327, Package_TO_SOT_THT:TO-92L_HandSolder, F.Cu at (265.4, 40.6)
- added Q_COUNT2: BC327, Package_TO_SOT_THT:TO-92L_HandSolder, F.Cu at (209.6, 41.9)
- added R_FLASH3: 2.2k 1/2W, Resistor_THT:R_Axial_DIN0207_L6.3mm_D2.5mm_P10.16mm_Horizontal, F.Cu at (259.1, 41.9)
- added R_FLASH4: 2.2k 1/2W, Resistor_THT:R_Axial_DIN0207_L6.3mm_D2.5mm_P10.16mm_Horizontal, F.Cu at (71.1, 105.4)
- added R_SW_PAPER5: 560ohm 1/2W, Resistor_THT:R_Axial_DIN0207_L6.3mm_D2.5mm_P10.16mm_Horizontal, F.Cu at (199.4, 38.1)
- CONN_BATT1, CONN_DC1, CONN_SW_BOTTOM1, CONN_SW_MIDDLE1, CONN_SW_SCISSOR1, CONN_SW_SHUTTER1, CONN_SW_UP1: footprint Connector_JST:JST_XH_S2B-XH-A_1x02_P2.50mm_Horizontal -> Connector_JST:JST_XH_S2B-XH-A-1_1x02_P2.50mm_Horizontal
- CONN_CEILING1, CONN_LGHT_PROCESS1, CONN_MARQUEE_WS2811, CONN_SERVO_ARM1, CONN_SW_PAP1, CONN_SW_PAP2, CONN_SW_PAP3, CONN_SW_PAP4, CONN_SW_ROT1, CONN_SW_ROT2, CONN_TEMP1: footprint Connector_JST:JST_XH_S3B-XH-A_1x03_P2.50mm_Horizontal -> Connector_JST:JST_XH_S3B-XH-A-1_1x03_P2.50mm_Horizontal
- CONN_COIN1, CONN_LUXSENSOR1, CONN_SEGMENT1, CONN_START1, CONN_STEP_EXIT1, CONN_STEP_PAPER1, CONN_STEP_ROT1, CONN_STEP_SCISSOR1, CONN_STEP_SHUTTER1: value Conn_01x04 -> JST_XH4; footprint Connector_JST:JST_XH_S4B-XH-A_1x04_P2.50mm_Horizontal -> Connector_JST:JST_XH_S4B-XH-A-1_1x04_P2.50mm_Horizontal
- CONN_MATRIX1: value Conn_01x05 -> JST_XH5; footprint Connector_JST:JST_XH_S5B-XH-A_1x05_P2.50mm_Horizontal -> Connector_JST:JST_XH_S5B-XH-A-1_1x05_P2.50mm_Horizontal
- C_ATTINY1: value 0.1uF -> 100nF
- C_AUX1, C_FLASH1: value 100uF -> 680uF; footprint Capacitor_THT:CP_Radial_D10.0mm_P5.00mm -> Capacitor_THT:CP_Radial_D8.0mm_P3.50mm
- C_CEILING1, C_DRV_PAPER1, C_DRV_SCISSOR1, C_DRV_SHUTTER1, C_LORA1, C_ROT1, C_SERVO_ARM1, C_STEP1: footprint Capacitor_THT:CP_Radial_D10.0mm_P5.00mm -> Capacitor_THT:CP_Radial_D6.3mm_P2.50mm
- C_LIGHT_PROCESS1: value 1000uF -> 100uF; footprint Capacitor_THT:CP_Radial_D10.0mm_P5.00mm -> Capacitor_THT:CP_Radial_D6.3mm_P2.50mm
- C_MARQUEE1: value 1000uF -> 680uF; footprint Capacitor_THT:CP_Radial_D10.0mm_P5.00mm -> Capacitor_THT:CP_Radial_D8.0mm_P3.50mm
- moved C_MEGA_PAPER1 244.5 mm to (17.8, 83.8), turned to 0 degrees
- moved H2 176.4 mm to (266.7, 25.4)
- moved H3 167.0 mm to (20.3, 33.0)
- moved H4 124.9 mm to (268.0, 113.0)
- moved H1 123.0 mm to (20.3, 113.0)
- moved CONN_DC1 84.5 mm to (157.5, 113.8)
- moved DRV_DC1 74.4 mm to (151.1, 85.1), turned to 180 degrees
- moved C_MATRIX1 61.9 mm to (240.0, 30.5), turned to 180 degrees
- moved U_RADIO1 49.4 mm to (178.3, 112.3)
- moved C_ATTINY1 32.0 mm to (83.8, 95.2), turned to 90 degrees
- moved R_SW_START1 29.3 mm to (185.4, 38.1), turned to 0 degrees
- moved CONN_SEGMENT1 21.6 mm to (256.5, 22.9)
- moved R_BATT2 20.6 mm to (168.9, 83.8), turned to 270 degrees
- moved CONN_MATRIX1 20.5 mm to (241.1, 22.9)
- moved R_SW_PAPER1 20.4 mm to (96.5, 38.1), turned to 0 degrees
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Connections:
- net /Camera/SERIAL_RX2 renamed /AtoB
- net /Paper/SERIAL_RX2 renamed /BtoA
- net BATT_PROBE renamed /Camera/BATT_PROBE
- net CEILING_PIXEL_PIN renamed /Camera/CEILING_PIXEL_PIN
- net COIN_PIN renamed /Camera/COIN_PIN
- net COIN_SEGMENT_CLK_PIN renamed /Camera/COIN_SEGMENT_CLK_PIN
- net COIN_SEGMENT_DIO_PIN renamed /Camera/COIN_SEGMENT_DIO_PIN
- net ENABLE_COIN_PIN renamed /Camera/ENABLE_COIN_PIN
- net ENABLE_MARQUEE renamed /Camera/ENABLE_MARQUEE
- net LED_MATRIX_CS_PIN renamed /Camera/LED_MATRIX_CS_PIN
- net LED_MATRIX_SCL_PIN renamed /Camera/LED_MATRIX_SCL_PIN
- net LED_MATRIX_SDI_PIN renamed /Camera/LED_MATRIX_SDI_PIN
- net LED_START_BTN_PIN renamed /Camera/LED_START_BTN_PIN
- net LORA_AUX renamed /Camera/LORA_AUX
- net LORA_M0 renamed /Camera/LORA_M0
- net LORA_M1 renamed /Camera/LORA_M1
- net LORA_RXD renamed /Camera/LORA_RXD
- net LORA_TXD renamed /Camera/LORA_TXD
- net PAPER_PIN_ENABLE renamed /Camera/PAPER_PIN_ENABLE
- net RADIO_INTERRUPT renamed /Camera/RADIO_INTERRUPT
- net RADIO_MISO renamed /Camera/RADIO_MISO
- net RADIO_MOSI renamed /Camera/RADIO_MOSI
- net RADIO_SCK renamed /Camera/RADIO_SCK
- net SCL_PIN renamed /Camera/SCL_PIN
- net SDA_PIN renamed /Camera/SDA_PIN
- net START_BTN_PIN renamed /Camera/START_BTN_PIN
- CONN_SW_PAP1 pad 2: PAPER_SWITCH1_PIN -> /Camera/PAPER_SWITCH1_PIN
- CONN_SW_PAP2 pad 2: PAPER_SWITCH2_PIN -> /Camera/PAPER_SWITCH2_PIN
- CONN_SW_PAP3 pad 2: PAPER_SWITCH3_PIN -> /Camera/PAPER_SWITCH3_PIN
- CONN_SW_PAP4 pad 2: PAPER_SWITCH4_PIN -> /Camera/PAPER_SWITCH4_PIN
- CONN_SW_SCISSOR1 pad 1: SCISSOR_ENDSTOP_PIN -> /Camera/SCISSOR_ENDSTOP_PIN
- CONN_SW_SHUTTER1 pad 1: SHUTTER_ENDSTOP_PIN -> /Camera/SHUTTER_ENDSTOP_PIN
- DRV_DC1 pad A: Net-(CONN_DC1-Pad2) -> Net-(CONN_DC1-Pad1)
- DRV_DC1 pad B: Net-(CONN_DC1-Pad1) -> Net-(CONN_DC1-Pad2)
- DRV_PAPER1 pad 10: PAPER_M0 -> /Camera/PAPER_M0
- DRV_PAPER1 pad 15: PAPER_PIN_STP -> /Camera/PAPER_PIN_STP
- DRV_PAPER1 pad 16: PAPER_PIN_DIR -> /Camera/PAPER_PIN_DIR
- DRV_SCISSOR1 pad 10: SCISSOR_M0 -> /Camera/SCISSOR_M0
- DRV_SCISSOR1 pad 15: SCISSOR_PIN_STP -> /Camera/SCISSOR_PIN_STP
- DRV_SCISSOR1 pad 16: SCISSOR_PIN_DIR -> /Camera/SCISSOR_PIN_DIR
- DRV_SCISSOR1 pad 9: SCISSOR_PIN_ENABLE -> /Camera/SCISSOR_PIN_ENABLE
- DRV_SHUTTER1 pad 10: SHUTTER_M0 -> /Camera/SHUTTER_M0
- DRV_SHUTTER1 pad 15: SHUTTER_PIN_STP -> /Camera/SHUTTER_PIN_STP
- DRV_SHUTTER1 pad 16: SHUTTER_PIN_DIR -> /Camera/SHUTTER_PIN_DIR
- DRV_SHUTTER1 pad 9: SHUTTER_PIN_ENABLE -> /Camera/SHUTTER_PIN_ENABLE
- LED_SW_PAPER1 pad 1: PAPER_SWITCH1_PIN -> /Camera/PAPER_SWITCH1_PIN
- LED_SW_PAPER2 pad 1: PAPER_SWITCH2_PIN -> /Camera/PAPER_SWITCH2_PIN
- LED_SW_PAPER3 pad 1: PAPER_SWITCH3_PIN -> /Camera/PAPER_SWITCH3_PIN
- LED_SW_PAPER4 pad 1: PAPER_SWITCH4_PIN -> /Camera/PAPER_SWITCH4_PIN
- LED_SW_SCISSOR1 pad 1: SCISSOR_ENDSTOP_PIN -> /Camera/SCISSOR_ENDSTOP_PIN
- LED_SW_SHUTTER1 pad 1: SHUTTER_ENDSTOP_PIN -> /Camera/SHUTTER_ENDSTOP_PIN
- MEGA_CAMERA1 pad D26: AUX_PIN -> /Camera/SHUTTER_ENDSTOP_PIN
- MEGA_CAMERA1 pad D27: FLASH_PIN -> /Camera/SCISSOR_ENDSTOP_PIN
- MEGA_CAMERA1 pad D28: (no net) -> /Camera/PAPER_SWITCH3_PIN
- MEGA_CAMERA1 pad D29: /Camera/ENABLE_5V -> /Camera/PAPER_SWITCH4_PIN
- MEGA_CAMERA1 pad D30: (no net) -> /Camera/PAPER_SWITCH1_PIN
- MEGA_CAMERA1 pad D31: (no net) -> /Camera/PAPER_SWITCH2_PIN
- MEGA_CAMERA1 pad D33: PAPER_M0 -> /Camera/PAPER_PIN_STP
- MEGA_CAMERA1 pad D34: PAPER_PIN_STP -> /Camera/PAPER_PIN_DIR
- MEGA_CAMERA1 pad D35: PAPER_PIN_DIR -> /Camera/PAPER_M0
- MEGA_CAMERA1 pad D36: SHUTTER_PIN_ENABLE -> /Camera/SHUTTER_M0
- MEGA_CAMERA1 pad D37: SHUTTER_M0 -> /Camera/SHUTTER_PIN_STP
- MEGA_CAMERA1 pad D38: SCISSOR_PIN_STP -> /Camera/SHUTTER_PIN_DIR
- MEGA_CAMERA1 pad D39: SCISSOR_PIN_DIR -> /Camera/SHUTTER_PIN_ENABLE
- MEGA_CAMERA1 pad D40: SCISSOR_PIN_ENABLE -> /Camera/SCISSOR_PIN_STP
- MEGA_CAMERA1 pad D41: SCISSOR_M0 -> /Camera/SCISSOR_PIN_DIR
- MEGA_CAMERA1 pad D42: SHUTTER_PIN_STP -> /Camera/SCISSOR_PIN_ENABLE
- MEGA_CAMERA1 pad D43: SHUTTER_PIN_DIR -> /Camera/SCISSOR_M0
- MEGA_CAMERA1 pad D44: SHUTTER_ENDSTOP_PIN -> /Camera/ENABLE_5V
- MEGA_CAMERA1 pad D45: SCISSOR_ENDSTOP_PIN -> /Camera/FLASH_PIN
- MEGA_CAMERA1 pad D46: PAPER_SWITCH1_PIN -> /Camera/AUX_PIN
- MEGA_CAMERA1 pad D47: PAPER_SWITCH2_PIN -> (no net)
- MEGA_CAMERA1 pad D48: PAPER_SWITCH3_PIN -> /Camera/RADIO_CE
- MEGA_CAMERA1 pad D49: PAPER_SWITCH4_PIN -> /Camera/RADIO_CSN
- MEGA_CAMERA1 pad D7: RADIO_CE -> (no net)
- MEGA_CAMERA1 pad D8: RADIO_CSN -> /Camera/COUNT_PIN
- MEGA_PAPER1 pad 5V: +5C -> (no net)
- MEGA_PAPER1 pad D39: (no net) -> /Paper/FAN_PIN
- R_FLASH1 pad 2: FLASH_PIN -> /Camera/FLASH_PIN
- R_FLASH2 pad 2: AUX_PIN -> /Camera/AUX_PIN
- U_RADIO1 pad 3: RADIO_CE -> /Camera/RADIO_CE
- U_RADIO1 pad 4: RADIO_CSN -> /Camera/RADIO_CSN
Routing:
- net +5V: track 0.00 -> 843.3 mm, vias 0 -> 6
- net +12V: track 0.00 -> 620.6 mm
- net /BtoA: track 0.00 -> 228.3 mm, vias 0 -> 2
- net /AtoB: track 0.00 -> 228.2 mm, vias 0 -> 2
- net /Camera/ORDER_INTERRUPT_PIN: track 0.00 -> 211.9 mm
- net +5C: track 0.00 -> 203.9 mm
- net /Camera/ENABLE_MARQUEE: track 0.00 -> 179.4 mm, vias 0 -> 1
- net /Camera/FLASH_PIN: track 0.00 -> 151.6 mm
- net /Camera/PAPER_SWITCH1_PIN: track 0.00 -> 135.3 mm
- net +3V3: track 0.00 -> 133.3 mm
- net /Camera/PAPER_SWITCH2_PIN: track 0.00 -> 126.8 mm
- net /Camera/RADIO_INTERRUPT: track 0.00 -> 118.0 mm
- net /Camera/PAPER_SWITCH3_PIN: track 0.00 -> 113.1 mm
- net /Camera/AUX_PIN: track 0.00 -> 107.8 mm, vias 0 -> 1
- net /Camera/PAPER_SWITCH4_PIN: track 0.00 -> 104.0 mm
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- added copper zone on F.Cu, net +12V
- added copper zone on F.Cu, net GND
Other:
- board size 270 x 90 mm -> 258.6 x 101.6 mm
- net class 2mm: trace_width 2 -> 1

Commit message: update
Routing:
- net /Camera/FLASH_PIN: track 151.6 -> 153.3 mm
Changed lines of the file:
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@@
     (thickness 1.6)
     (drawings 8)
-    (tracks 1086)
+    (tracks 1088)
     (zones 0)
     (modules 112)
@@
   (segment (start 128.27 72.39) (end 129.3953 72.39) (width 0.25) (layer B.Cu) (net 103))
   (via (at 193.3828 63.5) (size 0.8) (layers F.Cu B.Cu) (net 103))
-  (segment (start 223.52 82.55) (end 222.25 81.28) (width 0.25) (layer F.Cu) (net 104))
-  (segment (start 222.25 81.28) (end 216.5796 81.28) (width 0.25) (layer F.Cu) (net 104))
+  (segment (start 118.6003 66.675) (end 112.8853 72.39) (width 0.25) (layer F.Cu) (net 104))
+  (segment (start 112.8853 72.39) (end 111.76 72.39) (width 0.25) (layer F.Cu) (net 104))
+  (segment (start 137.795 66.675) (end 118.6003 66.675) (width 0.25) (layer F.Cu) (net 104))
+  (segment (start 157.48 51.435) (end 153.035 51.435) (width 0.25) (layer F.Cu) (net 104))
+  (segment (start 164.5533 58.5083) (end 157.48 51.435) (width 0.25) (layer F.Cu) (net 104))
+  (segment (start 164.5533 65.8364) (end 164.5533 58.5083) (width 0.25) (layer F.Cu) (net 104))
   (segment (start 216.5796 81.28) (end 200.8746 65.575) (width 0.25) (layer F.Cu) (net 104))
-  (segment (start 200.8746 65.575) (end 200.8746 63.4422) (width 0.25) (layer F.Cu) (net 104))
+  (segment (start 165.8446 67.1277) (end 164.5533 65.8364) (width 0.25) (layer F.Cu) (net 104))
+  (segment (start 223.52 82.55) (end 222.25 81.28) (width 0.25) (layer F.Cu) (net 104))
   (segment (start 200.8746 63.4422) (end 191.7814 54.349) (width 0.25) (layer F.Cu) (net 104))
+  (segment (start 200.8746 65.575) (end 200.8746 63.4422) (width 0.25) (layer F.Cu) (net 104))
   (segment (start 191.7814 54.349) (end 173.9093 54.349) (width 0.25) (layer F.Cu) (net 104))
+  (segment (start 153.035 51.435) (end 137.795 66.675) (width 0.25) (layer F.Cu) (net 104))
   (segment (start 173.9093 54.349) (end 172.8738 55.3845) (width 0.25) (layer F.Cu) (net 104))
+  (segment (start 222.25 81.28) (end 216.5796 81.28) (width 0.25) (layer F.Cu) (net 104))
   (segment (start 172.8738 55.3845) (end 172.8738 62.0007) (width 0.25) (layer F.Cu) (net 104))
-  (segment (start 172.8738 62.0007) (end 167.7468 67.1277) (width 0.25) (layer F.Cu) (net 104))
   (segment (start 167.7468 67.1277) (end 165.8446 67.1277) (width 0.25) (layer F.Cu) (net 104))
-  (segment (start 165.8446 67.1277) (end 164.5533 65.8364) (width 0.25) (layer F.Cu) (net 104))
-  (segment (start 164.5533 65.8364) (end 164.5533 60.037) (width 0.25) (layer F.Cu) (net 104))
-  (segment (start 164.5533 60.037) (end 156.9778 52.4615) (width 0.25) (layer F.Cu) (net 104))
-  (segment (start 156.9778 52.4615) (end 132.8138 52.4615) (width 0.25) (layer F.Cu) (net 104))
-  (segment (start 132.8138 52.4615) (end 112.8853 72.39) (width 0.25) (layer F.Cu) (net 104))
-  (segment (start 111.76 72.39) (end 112.8853 72.39) (width 0.25) (layer F.Cu) (net 104))
+  (segment (start 172.8738 62.0007) (end 167.7468 67.1277) (width 0.25) (layer F.Cu) (net 104))
   (segment (start 168.91 83.82) (end 177.3346 92.2446) (width 0.25) (layer F.Cu) (net 105))
   (segment (start 177.3346 92.2446) (end 221.2687 92.2446) (width 0.25) (layer F.Cu) (net 105))

Commit message: pcb finalized
Parts:
- removed CONN_SW_MIDDLE1: JST_XH2, Connector_JST:JST_XH_S2B-XH-A-1_1x02_P2.50mm_Horizontal
- removed LED_SW_MIDDLE1: LED 3mm, LED_THT:LED_D3.0mm
- removed R_SW_MIDDLE1, R_SW_PAPER5: 560ohm 1/2W, Resistor_THT:R_Axial_DIN0207_L6.3mm_D2.5mm_P10.16mm_Horizontal
- added J_AUX_CAM1: Conn_01x10, Connector_PinHeader_2.54mm:PinHeader_1x05_P2.54mm_Vertical, F.Cu at (259.7, 43.2)
- added J_AUX_PAPER1: Conn_01x10, Connector_PinHeader_2.54mm:PinHeader_1x10_P2.54mm_Vertical, F.Cu at (18.4, 38.7)
- added R_LED_START1: 560ohm, Resistor_THT:R_Axial_DIN0207_L6.3mm_D2.5mm_P10.16mm_Horizontal, F.Cu at (200.7, 38.7)
- R_BATT1: value 20k1/2W -> 20k
- R_BATT2: value 10k 1/2W -> 10k
- R_FLASH1, R_FLASH2, R_FLASH3, R_FLASH4, R_START1: value 2.2k 1/2W -> 2.2k
- R_MARQUEE1: value 430ohm 1/2W -> 430ohm
- R_RXD_LORA1, R_TXD_LORA1: value 4.7k 1/2W -> 4.7k
- R_SW_BOTTOM1, R_SW_PAPER1, R_SW_PAPER2, R_SW_PAPER3, R_SW_PAPER4, R_SW_ROT1, R_SW_ROT2, R_SW_SCISSOR1, R_SW_SHUTTER1, R_SW_START1, R_SW_UP1: value 560ohm 1/2W -> 560ohm
- U_MARQUEE1: value ATtiny85-20PU -> ATtiny85
- moved R_SW_ROT2 14.8 mm to (49.5, 52.1)
- moved R_SW_ROT1 14.8 mm to (35.6, 52.1)
- moved R_SW_UP1 14.8 mm to (63.5, 52.1)
- moved C_CAMERA_5V2 13.3 mm to (266.7, 31.8), turned to 270 degrees
- moved LED_SW_ROT2 10.9 mm to (47.6, 31.8)
- moved LED_SW_UP1 10.9 mm to (57.8, 31.8)
- moved CONN_SW_UP1 10.2 mm to (58.4, 22.6)
- moved CONN_SW_ROT1 10.2 mm to (35.5, 22.6)
- moved CONN_SW_ROT2 10.2 mm to (48.2, 22.6)
- moved H3 9.55 mm to (21.0, 23.5)
- moved LED_SW_ROT1 7.73 mm to (34.3, 31.8)
- moved CONN_COUNT1 7.65 mm to (271.1, 33.0), turned to 0 degrees
- moved R_FLASH3 7.41 mm to (255.3, 35.6), turned to 180 degrees
- moved Q_COUNT1 5.99 mm to (262.3, 35.6)
- moved C_DRV_SCISSOR1 1.42 mm to (264.2, 109.2)
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- renumbered Q_COUNT2 to Q_START1
Connections:
- MEGA_CAMERA1 pad A13: (no net) -> /Camera/A13
- MEGA_CAMERA1 pad A14: (no net) -> /Camera/A14
- MEGA_CAMERA1 pad D47: (no net) -> /Camera/D47
- MEGA_CAMERA1 pad D53: (no net) -> /Camera/D53
- MEGA_CAMERA1 pad D7: (no net) -> /Camera/D7
- MEGA_PAPER1 pad A4: (no net) -> /Paper/A4
- MEGA_PAPER1 pad A5: (no net) -> /Paper/A5
- MEGA_PAPER1 pad D35: SPIDER_UPDOWN_PIN_ENDSTOP_MIDDLE -> (no net)
- MEGA_PAPER1 pad D38: (no net) -> /Paper/D38
- MEGA_PAPER1 pad D40: (no net) -> /Paper/D40
- MEGA_PAPER1 pad D41: (no net) -> /Paper/D41
- MEGA_PAPER1 pad D42: (no net) -> /Paper/D42
- MEGA_PAPER1 pad D43: (no net) -> /Paper/D43
- MEGA_PAPER1 pad D47: (no net) -> /Paper/D47
- MEGA_PAPER1 pad D48: (no net) -> /Paper/D48
- MEGA_PAPER1 pad D49: (no net) -> /Paper/D49
Routing:
- net /Camera/D47: track 0.00 -> 146.6 mm
- net /Camera/A14: track 0.00 -> 89.1 mm
- net /Paper/D38: track 0.00 -> 61.6 mm
- net /Camera/D53: track 0.00 -> 56.2 mm, vias 0 -> 1
- net /Paper/D40: track 0.00 -> 53.1 mm
- net /Paper/D47: track 0.00 -> 52.3 mm, vias 0 -> 1
- net /Camera/A13: track 0.00 -> 50.6 mm, vias 0 -> 1
- net /Paper/D42: track 0.00 -> 43.8 mm
- net /Paper/D48: track 0.00 -> 40.6 mm, vias 0 -> 1
- net /Paper/D41: track 0.00 -> 40.6 mm
- net /Paper/D43: track 0.00 -> 37.5 mm
- net /Paper/D49: track 0.00 -> 32.2 mm, vias 0 -> 2
- net +5V: track 843.3 -> 872.0 mm
- net SPIDER_UPDOWN_PIN_ENDSTOP_MIDDLE: track 26.3 -> 0.00 mm
- net /Paper/A4: track 0.00 -> 21.8 mm
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Other:
- board text added: "+"
- board text added: "12V"
- board text added: "5V"
- board text added: "A13"
- board text added: "A14"
- board text added: "A4"
- board text added: "A5"
- board text added: "CLK"
- board text added: "CS"
- board text added: "D38"
- board text added: "D40"
- board text added: "D41"
- board text added: "D42"
- board text added: "D43"
- board text added: "D47"
- board text added: "D48"
- board text added: "D49"
- board text added: "D53"
- board text added: "D7"
- board text added: "DIO"
- board text added: "ENB"
- board text added: "GND"
- board text added: "INT"
- board text added: "No filter booth PCB V0.Gilou"
- board text added: "SCL"
- board text added: "SDA"
- board text added: "SDL"
- board text added: "SW"

Commit message: Update, code for the pcb version.
Parts:
- moved C_AUX3 3.17 mm to (74.3, 90.2), turned to 0 degrees
Connections:
- C_AUX3 pad 1: GND -> +12V
- C_AUX3 pad 2: +12V -> GND
Changed lines of the file:
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@@
     (add_net "Net-(CONN_STEP_SHUTTER1-Pad3)")
     (add_net "Net-(CONN_STEP_SHUTTER1-Pad4)")
+    (add_net "Net-(DRV_EXIT1-Pad2)")
+    (add_net "Net-(DRV_PAPER1-Pad2)")
+    (add_net "Net-(DRV_ROT1-Pad2)")
+    (add_net "Net-(DRV_SCISSOR1-Pad2)")
+    (add_net "Net-(DRV_SHUTTER1-Pad2)")
     (add_net "Net-(LED_SW_BOTTOM1-Pad2)")
     (add_net "Net-(LED_SW_PAPER1-Pad2)")
@@
     (add_net "Net-(LED_SW_START1-Pad2)")
     (add_net "Net-(LED_SW_UP1-Pad2)")
+    (add_net "Net-(MEGA_CAMERA1-PadA0)")
+    (add_net "Net-(MEGA_CAMERA1-PadA1)")
+    (add_net "Net-(MEGA_CAMERA1-PadA10)")
+    (add_net "Net-(MEGA_CAMERA1-PadA11)")
+    (add_net "Net-(MEGA_CAMERA1-PadA12)")
+    (add_net "Net-(MEGA_CAMERA1-PadA2)")
+    (add_net "Net-(MEGA_CAMERA1-PadA3)")
+    (add_net "Net-(MEGA_CAMERA1-PadA4)")
+    (add_net "Net-(MEGA_CAMERA1-PadA5)")
+    (add_net "Net-(MEGA_CAMERA1-PadA6)")
+    (add_net "Net-(MEGA_CAMERA1-PadA7)")
+    (add_net "Net-(MEGA_CAMERA1-PadA8)")
+    (add_net "Net-(MEGA_CAMERA1-PadA9)")
+    (add_net "Net-(MEGA_CAMERA1-PadAREF)")
+    (add_net "Net-(MEGA_CAMERA1-PadMISO)")
+    (add_net "Net-(MEGA_CAMERA1-PadMOSI)")
+    (add_net "Net-(MEGA_CAMERA1-PadRESET)")
+    (add_net "Net-(MEGA_CAMERA1-PadRST)")
+    (add_net "Net-(MEGA_CAMERA1-PadRX)")
+    (add_net "Net-(MEGA_CAMERA1-PadSCK)")
+    (add_net "Net-(MEGA_CAMERA1-PadTX)")
+    (add_net "Net-(MEGA_CAMERA1-PadVCC)")
     (add_net "Net-(MEGA_PAPER1-Pad3V3)")
+    (add_net "Net-(MEGA_PAPER1-Pad5V)")
+    (add_net "Net-(MEGA_PAPER1-PadA0)")
+    (add_net "Net-(MEGA_PAPER1-PadA1)")
+    (add_net "Net-(MEGA_PAPER1-PadA10)")
+    (add_net "Net-(MEGA_PAPER1-PadA11)")
+    (add_net "Net-(MEGA_PAPER1-PadA12)")
+    (add_net "Net-(MEGA_PAPER1-PadA13)")
+    (add_net "Net-(MEGA_PAPER1-PadA14)")
+    (add_net "Net-(MEGA_PAPER1-PadA15)")
+    (add_net "Net-(MEGA_PAPER1-PadA2)")
+    (add_net "Net-(MEGA_PAPER1-PadA3)")
+    (add_net "Net-(MEGA_PAPER1-PadA6)")
+    (add_net "Net-(MEGA_PAPER1-PadA7)")
+    (add_net "Net-(MEGA_PAPER1-PadA8)")
+    (add_net "Net-(MEGA_PAPER1-PadA9)")
+    (add_net "Net-(MEGA_PAPER1-PadAREF)")
+    (add_net "Net-(MEGA_PAPER1-PadD16)")
+    (add_net "Net-(MEGA_PAPER1-PadD17)")
+    (add_net "Net-(MEGA_PAPER1-PadD18)")
+    (add_net "Net-(MEGA_PAPER1-PadD19)")
+    (add_net "Net-(MEGA_PAPER1-PadD20)")
+    (add_net "Net-(MEGA_PAPER1-PadD21)")
+    (add_net "Net-(MEGA_PAPER1-PadD22)")
+    (add_net "Net-(MEGA_PAPER1-PadD23)")
+    (add_net "Net-(MEGA_PAPER1-PadD24)")
+    (add_net "Net-(MEGA_PAPER1-PadD25)")
+    (add_net "Net-(MEGA_PAPER1-PadD26)")
+    (add_net "Net-(MEGA_PAPER1-PadD27)")
+    (add_net "Net-(MEGA_PAPER1-PadD28)")
+    (add_net "Net-(MEGA_PAPER1-PadD29)")
+    (add_net "Net-(MEGA_PAPER1-PadD3)")
+    (add_net "Net-(MEGA_PAPER1-PadD30)")
+    (add_net "Net-(MEGA_PAPER1-PadD31)")
+    (add_net "Net-(MEGA_PAPER1-PadD50)")
+    (add_net "Net-(MEGA_PAPER1-PadD51)")
+    (add_net "Net-(MEGA_PAPER1-PadD52)")
+    (add_net "Net-(MEGA_PAPER1-PadD53)")
+    (add_net "Net-(MEGA_PAPER1-PadMISO)")
+    (add_net "Net-(MEGA_PAPER1-PadMOSI)")
+    (add_net "Net-(MEGA_PAPER1-PadRESET)")
+    (add_net "Net-(MEGA_PAPER1-PadRST)")
+    (add_net "Net-(MEGA_PAPER1-PadRX)")
+    (add_net "Net-(MEGA_PAPER1-PadSCK)")
+    (add_net "Net-(MEGA_PAPER1-PadTX)")
+    (add_net "Net-(MEGA_PAPER1-PadVCC)")
     (add_net "Net-(Q_AUX1-Pad1)")
     (add_net "Net-(Q_AUX2-Pad1)")
@@
     (add_net "Net-(Q_START1-Pad2)")
     (add_net "Net-(R_MARQUEE1-Pad1)")
+    (add_net "Net-(URTC1-PadND)")
+    (add_net "Net-(U_MARQUEE1-Pad1)")
+    (add_net "Net-(U_MARQUEE1-Pad3)")
+    (add_net "Net-(U_MARQUEE1-Pad5)")
+    (add_net "Net-(U_MARQUEE1-Pad7)")
+    (add_net "Net-(U_STEP_DOWN_5V1-PadFB)")
+    (add_net "Net-(U_STEP_DOWN_5V1-PadPG)")
     (add_net ROT_M0)
     (add_net SERVO_ARM)
@@
     (add_net SPIDER_UPDOWN_PIN_DIR)
     (add_net SPIDER_UPDOWN_PIN_ENDSTOP_BOTTOM)
+    (add_net SPIDER_UPDOWN_PIN_ENDSTOP_MIDDLE)
     (add_net SPIDER_UPDOWN_PIN_ENDSTOP_UP)
     (add_net SPIDER_UPDOWN_PIN_PWM)
@@
   )
   (module Capacitor_THT:CP_Radial_D8.0mm_P3.50mm (layer F.Cu)
-    (at 77.47 90.17 180)
+    (at 74.295 90.17)
     (descr "CP, Radial series, Radial, pin pitch=3.50mm, , diameter=8mm, Electrolytic Capacitor")
     (tags "CP Radial series Radial pin pitch 3.50mm  diameter 8mm Electrolytic Capacitor")
@@
     (fp_circle (center 1.75 0) (end 5.87 0) (layer F.SilkS) (width 0.12))
     (fp_circle (center 1.75 0) (end 5.75 0) (layer F.Fab) (width 0.1))
-    (pad 2 thru_hole circle (at 3.5 0 180) (size 1.6 1.6) (drill 0.8) (layers *.Cu *.Mask)
-      (net 2 +12V))
-    (pad 1 thru_hole rect (at 0 0 180) (size 1.6 1.6) (drill 0.8) (layers *.Cu *.Mask)
+    (pad 2 thru_hole circle (at 3.5 0) (size 1.6 1.6) (drill 0.8) (layers *.Cu *.Mask)
       (net 1 GND))
+    (pad 1 thru_hole rect (at 0 0) (size 1.6 1.6) (drill 0.8) (layers *.Cu *.Mask)
+      (net 2 +12V))
     (model ${KISYS3DMOD}/Capacitor_THT.3dshapes/CP_Radial_D8.0mm_P3.50mm.wrl
       (at (xyz 0 0 0))
@@
   (segment (start 44.45 104.14) (end 44.45 110.49) (width 2) (layer F.Cu) (net 2))
   (segment (start 271.78 49.53) (end 271.78 52.07) (width 1) (layer F.Cu) (net 2))
-  (segment (start 73.97 90.17) (end 73.97 92.4) (width 2) (layer F.Cu) (net 2))
-  (segment (start 73.97 92.4) (end 64.77 101.6) (width 2) (layer F.Cu) (net 2))
   (segment (start 78.74 113.76) (end 78.74 116.84) (width 2) (layer F.Cu) (net 2))
   (segment (start 64.77 101.6) (end 67.31 104.14) (width 2) (layer F.Cu) (net 2))
@@
   (segment (start 264.16 109.22) (end 265.43 109.22) (width 2) (layer F.Cu) (net 2))
   (segment (start 265.43 109.22) (end 270.51 104.14) (width 2) (layer F.Cu) (net 2))
+  (segment (start 74.295 92.075) (end 64.77 101.6) (width 2) (layer F.Cu) (net 2))
+  (segment (start 74.295 90.17) (end 74.295 92.075) (width 2) (layer F.Cu) (net 2))
   (segment (start 212.09 102.87) (end 212.09 106.68) (width 1) (layer F.Cu) (net 3))
   (segment (start 212.09 106.68) (end 211.995 106.68) (width 1) (layer F.Cu) (net 3))
