File: hardware/kicad/paper.sch (KiCad schematic (older format))
At the start: 34 parts

Commit message: pcb finalized
Parts:
- removed CONN_SW_MIDDLE1: JST_XH2, Connector_JST:JST_XH_S2B-XH-A-1_1x02_P2.50mm_Horizontal, symbol 1nofilterbooth:Conn_01x02-Connector_Generic
- removed LED_SW_MIDDLE1: LED 3mm, LED_THT:LED_D3.0mm, symbol 1nofilterbooth:LED_Small-Device
- removed R_SW_MIDDLE1: 560ohm 1/2W, Resistor_THT:R_Axial_DIN0207_L6.3mm_D2.5mm_P10.16mm_Horizontal, symbol 1nofilterbooth:R_Small-Device
- added J_AUX_PAPER1: Conn_01x10, Connector_PinHeader_2.54mm:PinHeader_1x10_P2.54mm_Vertical, symbol Connector_Generic:Conn_01x10
- R_FLASH4: value 2.2k 1/2W -> 2.2k
- R_SW_BOTTOM1, R_SW_ROT1, R_SW_ROT2, R_SW_UP1: value 560ohm 1/2W -> 560ohm
Connections:
- net A4: now reaches MEGA_PAPER1.A4
- net A4: now also J_AUX_PAPER1.1 (Pin_1)
- net A5: now reaches MEGA_PAPER1.A5
- net A5: now also J_AUX_PAPER1.2 (Pin_2)
- net D38: now reaches MEGA_PAPER1.D38
- net D38: now also J_AUX_PAPER1.3 (Pin_3)
- net D40: now reaches MEGA_PAPER1.D40
- net D40: now also J_AUX_PAPER1.4 (Pin_4)
- net D41: now reaches MEGA_PAPER1.D41
- net D41: now also J_AUX_PAPER1.5 (Pin_5)
- net D42: now reaches MEGA_PAPER1.D42
- net D42: now also J_AUX_PAPER1.6 (Pin_6)
- net D43: now reaches MEGA_PAPER1.D43
- net D43: now also J_AUX_PAPER1.7 (Pin_7)
- net D47: now reaches MEGA_PAPER1.D47
- net D47: now also J_AUX_PAPER1.8 (Pin_8)
- net D48: now reaches MEGA_PAPER1.D48
- net D48: now also J_AUX_PAPER1.9 (Pin_9)
- net D49: now reaches MEGA_PAPER1.D49
- net D49: now also J_AUX_PAPER1.10 (Pin_10)
- no-connect marks 60 -> 50
Changed lines of the file:
@@
 AR Path="/5E432787/5E451679" Ref="R_SW_ROT1"  Part="1"
 F 0 "R_SW_ROT1" V 9379 925 50  0000 C CNN
-F 1 "560ohm 1/2W" V 9470 925 50  0000 C CNN
+F 1 "560ohm" V 9470 925 50  0000 C CNN
 F 2 "Resistor_THT:R_Axial_DIN0207_L6.3mm_D2.5mm_P10.16mm_Horizontal" H 9575 925 50  0001 C CNN
 F 3 "~" H 9575 925 50  0001 C CNN
@@
 AR Path="/5E432787/5E453007" Ref="R_SW_ROT2"  Part="1"
 F 0 "R_SW_ROT2" V 9329 1775 50  0000 C CNN
-F 1 "560ohm 1/2W" V 9420 1775 50  0000 C CNN
+F 1 "560ohm" V 9420 1775 50  0000 C CNN
 F 2 "Resistor_THT:R_Axial_DIN0207_L6.3mm_D2.5mm_P10.16mm_Horizontal" H 9525 1775 50  0001 C CNN
 F 3 "~" H 9525 1775 50  0001 C CNN
@@
 AR Path="/5E432787/5E45951E" Ref="R_SW_UP1"  Part="1"
 F 0 "R_SW_UP1" V 9504 2725 50  0000 C CNN
-F 1 "560ohm 1/2W" V 9595 2725 50  0000 C CNN
+F 1 "560ohm" V 9595 2725 50  0000 C CNN
 F 2 "Resistor_THT:R_Axial_DIN0207_L6.3mm_D2.5mm_P10.16mm_Horizontal" H 9700 2725 50  0001 C CNN
 F 3 "~" H 9700 2725 50  0001 C CNN
@@
 F 3 "" H 9800 2725 50  0001 C CNN
 	1    9800 2725
-	0    1    1    0
-$EndComp
-$Comp
-L 1nofilterbooth:GND-power #PWR?
-U 1 1 5E45AF2B
-P 9975 4050
-AR Path="/5E3BF423/5E45AF2B" Ref="#PWR?"  Part="1"
-AR Path="/5E432787/5E45AF2B" Ref="#PWR0194"  Part="1"
-F 0 "#PWR0194" H 9975 3800 50  0001 C CNN
-F 1 "GND" V 9980 3922 50  0000 R CNN
-F 2 "" H 9975 4050 50  0001 C CNN
-F 3 "" H 9975 4050 50  0001 C CNN
-	1    9975 4050
-	0    1    1    0
-$EndComp
-Wire Wire Line
-	9375 3950 9675 3950
-Text GLabel 9375 3950 0    50   Input ~ 0
-SPIDER_UPDOWN_PIN_ENDSTOP_MIDDLE
-$Comp
-L 1nofilterbooth:Conn_01x02-Connector_Generic CONN_SW_UP?
-U 1 1 5E45AF37
-P 10175 3950
-AR Path="/5E45AF37" Ref="CONN_SW_UP?"  Part="1"
-AR Path="/5E3BF423/5E45AF37" Ref="CONN_SW_UP?"  Part="1"
-AR Path="/5E432787/5E45AF37" Ref="CONN_SW_MIDDLE1"  Part="1"
-F 0 "CONN_SW_MIDDLE1" H 10255 3942 50  0000 L CNN
-F 1 "JST_XH2" H 10255 3851 50  0000 L CNN
-F 2 "Connector_JST:JST_XH_S2B-XH-A-1_1x02_P2.50mm_Horizontal" H 10175 3950 50  0001 C CNN
-F 3 "~" H 10175 3950 50  0001 C CNN
-	1    10175 3950
-	1    0    0    -1
-$EndComp
-$Comp
-L 1nofilterbooth:LED_Small-Device LED_SW_UP?
-U 1 1 5E45AF41
-P 9675 3850
-AR Path="/5E3BF423/5E45AF41" Ref="LED_SW_UP?"  Part="1"
-AR Path="/5E432787/5E45AF41" Ref="LED_SW_MIDDLE1"  Part="1"
-F 0 "LED_SW_MIDDLE1" V 9675 4525 50  0000 R CNN
-F 1 "LED 3mm" V 9750 4225 50  0000 R CNN
-F 2 "LED_THT:LED_D3.0mm" V 9675 3850 50  0001 C CNN
-F 3 "~" V 9675 3850 50  0001 C CNN
-	1    9675 3850
-	0    -1   -1   0
-$EndComp
-Connection ~ 9675 3950
-Wire Wire Line
-	9675 3950 9975 3950
-$Comp
-L 1nofilterbooth:R_Small-Device R_SW_UP?
-U 1 1 5E45AF4D
-P 9775 3750
-AR Path="/5E3BF423/5E45AF4D" Ref="R_SW_UP?"  Part="1"
-AR Path="/5E432787/5E45AF4D" Ref="R_SW_MIDDLE1"  Part="1"
-F 0 "R_SW_MIDDLE1" V 9579 3750 50  0000 C CNN
-F 1 "560ohm 1/2W" V 9670 3750 50  0000 C CNN
-F 2 "Resistor_THT:R_Axial_DIN0207_L6.3mm_D2.5mm_P10.16mm_Horizontal" H 9775 3750 50  0001 C CNN
-F 3 "~" H 9775 3750 50  0001 C CNN
-	1    9775 3750
-	0    1    1    0
-$EndComp
-$Comp
-L 1nofilterbooth:+5V-power #PWR?
-U 1 1 5E45AF57
-P 9875 3750
-AR Path="/5E3BF423/5E45AF57" Ref="#PWR?"  Part="1"
-AR Path="/5E432787/5E45AF57" Ref="#PWR0195"  Part="1"
-F 0 "#PWR0195" H 9875 3600 50  0001 C CNN
-F 1 "+5V" V 9890 3878 50  0000 L CNN
-F 2 "" H 9875 3750 50  0001 C CNN
-F 3 "" H 9875 3750 50  0001 C CNN
-	1    9875 3750
 	0    1    1    0
 $EndComp
@@
 AR Path="/5E432787/5E45F215" Ref="R_SW_BOTTOM1"  Part="1"
 F 0 "R_SW_BOTTOM1" V 9579 4550 50  0000 C CNN
-F 1 "560ohm 1/2W" V 9670 4550 50  0000 C CNN
+F 1 "560ohm" V 9670 4550 50  0000 C CNN
 F 2 "Resistor_THT:R_Axial_DIN0207_L6.3mm_D2.5mm_P10.16mm_Horizontal" H 9775 4550 50  0001 C CNN
 F 3 "~" H 9775 4550 50  0001 C CNN
@@
 NoConn ~ 6225 1775
 NoConn ~ 6225 1875
-NoConn ~ 6225 1975
-NoConn ~ 6225 2075
 NoConn ~ 6225 2175
 NoConn ~ 6225 2275
@@
 NoConn ~ 6225 2975
 NoConn ~ 6225 3075
-NoConn ~ 6225 3775
-NoConn ~ 6225 3975
-NoConn ~ 6225 4075
-NoConn ~ 6225 4175
-NoConn ~ 6225 4275
-NoConn ~ 6225 4675
-NoConn ~ 6225 4775
-NoConn ~ 6225 4875
 NoConn ~ 6225 4975
 NoConn ~ 6225 5075
@@
 AR Path="/5E432787/5E496055" Ref="R_FLASH4"  Part="1"
 F 0 "R_FLASH4" V 9979 5825 50  0000 C CNN
-F 1 "2.2k 1/2W" V 10070 5825 50  0000 C CNN
+F 1 "2.2k" V 10070 5825 50  0000 C CNN
 F 2 "Resistor_THT:R_Axial_DIN0207_L6.3mm_D2.5mm_P10.16mm_Horizontal" H 10175 5825 50  0001 C CNN
 F 3 "~" H 10175 5825 50  0001 C CNN
@@
 NoConn ~ 5225 1875
 NoConn ~ 5225 1775
+$Comp
+L Connector_Generic:Conn_01x10 J_AUX_PAPER1
+U 1 1 5E4C98B4
+P 1475 6775
+F 0 "J_AUX_PAPER1" V 1692 6721 50  0000 C CNN
+F 1 "Conn_01x10" V 1601 6721 50  0000 C CNN
+F 2 "Connector_PinHeader_2.54mm:PinHeader_1x10_P2.54mm_Vertical" H 1475 6775 50  0001 C CNN
+F 3 "~" H 1475 6775 50  0001 C CNN
+	1    1475 6775
+	0    -1   -1   0
+$EndComp
+Text Label 1075 6975 3    50   ~ 0
+A4
+Text Label 1175 6975 3    50   ~ 0
+A5
+Text Label 6225 1975 0    50   ~ 0
+A4
+Text Label 6225 2075 0    50   ~ 0
+A5
+Text Label 6225 4675 0    50   ~ 0
+D47
+Text Label 6225 3775 0    50   ~ 0
+D38
+Text Label 6225 3975 0    50   ~ 0
+D40
+Text Label 6225 4075 0    50   ~ 0
+D41
+Text Label 6225 4175 0    50   ~ 0
+D42
+Text Label 6225 4275 0    50   ~ 0
+D43
+Text Label 6225 4775 0    50   ~ 0
+D48
+Text Label 6225 4875 0    50   ~ 0
+D49
+Text Label 1275 6975 3    50   ~ 0
+D38
+Text Label 1375 6975 3    50   ~ 0
+D40
+Text Label 1475 6975 3    50   ~ 0
+D41
+Text Label 1575 6975 3    50   ~ 0
+D42
+Text Label 1675 6975 3    50   ~ 0
+D43
+Text Label 1775 6975 3    50   ~ 0
+D47
+Text Label 1875 6975 3    50   ~ 0
+D48
+Text Label 1975 6975 3    50   ~ 0
+D49
 $EndSCHEMATC

Commit message: Update, code for the pcb version.
Connections:
- net +12V: now also C_AUX3.1; no longer C_AUX3.2
- net GND: now also C_AUX3.2; no longer C_AUX3.1
Changed lines of the file:
@@
 F 3 "~" H 9650 5550 50  0001 C CNN
 	1    9650 5550
-	-1   0    0    1
+	1    0    0    -1
 $EndComp
 $Comp
